File: TestBoardv1/BusPirate-ultra-testboard.v1.0.sch (EAGLE design)
At the start: 24 parts, among them J1 CON_HEADER_1X10-RIGHT_ANGLED_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

Commit message: fix testboard IO header to match v1b, created gerbers
Parts:
- added LED15, LED16: (no value), dp_devices.v6:LED-0805
Connections:
- removed net 3V3: J1.3, J1.4, LED10.A, LED12.A, LED2.A, LED4.A, LED6.A, LED8.A, R7.1
- removed net 5V0: J1.2, R8.1
- removed net ADC_DAC: J1.5, R6.1
- removed net AUX: J1.6, R5.1
- removed net CLOCK: J1.9, R2.1
- removed net CS: J1.7, R4.1
- removed net MISO: J1.8, R3.1
- removed net MOSI: J1.10, R1.1
- new net BPIO0: J1.1, R8.1
- new net BPIO1: J1.2, R7.1
- new net BPIO2: J1.3, R6.1
- new net BPIO3: J1.4, R5.1
- new net BPIO4: J1.5, R4.1
- new net BPIO5: J1.6, R3.1
- new net BPIO6: J1.7, R2.1
- new net BPIO7: J1.8, R1.1
- new net VOUT: J1.9, LED10.A, LED12.A, LED15.A, LED16.A, LED2.A, LED4.A, LED6.A, LED8.A
- net GND: now also J1.10; no longer J1.1
- net N$7: now also LED15.C
- net N$8: now also LED16.C
Other:
- note added: "BPIO0"
- note added: "BPIO1"
- note added: "BPIO2"
- note added: "BPIO3"
- note added: "BPIO4"
- note added: "BPIO5"
- note added: "BPIO6"
- note added: "BPIO7"
- note added: "Vout"
- note removed: "ADC/DAC"
- note removed: "AUX"
- note removed: "CLOCK"
- note removed: "CS"
- note removed: "MISO"
- note removed: "MOSI"
- note removed: "SWV33"
- note removed: "SWV50"
- note removed: "VEXTERN"
- moved on the sheet: R7, R8

Commit message: added vout and GND test point. add LED status to vout
Parts:
- added J2: CON_HEADER_1X02-PTH, dp_devices.v6:CON_HEADER_1X02-PTH
- added LED17: (no value), dp_devices.v6:LED-0805
- added R9: 1k1, dp_devices.v6:RESISTOR-0603
Connections:
- new net N$9: LED17.A, R9.2
- net GND: now also J2.2, LED17.C
- net VOUT: now also J2.1, R9.1
Other:
- note added: "TEST POINT"
Changed lines of the file:
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@@
 <?xml version="1.0" encoding="utf-8"?>
 <!DOCTYPE eagle SYSTEM "eagle.dtd">
-<eagle version="9.4.2">
+<eagle version="9.1.3">
 <drawing>
 <settings>
@@
 <part name="LED15" library="dp_devices.v6" deviceset="LED" device="-0805"/>
 <part name="LED16" library="dp_devices.v6" deviceset="LED" device="-0805"/>
+<part name="LED17" library="dp_devices.v6" deviceset="LED" device="-0805"/>
+<part name="SUPPLY10" library="supply2" library_urn="urn:adsk.eagle:library:372" deviceset="DGND" device=""/>
+<part name="J2" library="dp_devices.v6" deviceset="CON_HEADER_1X02" device="-PTH"/>
+<part name="SUPPLY11" library="supply2" library_urn="urn:adsk.eagle:library:372" deviceset="DGND" device=""/>
+<part name="R9" library="dp_devices.v6" deviceset="RESISTOR" device="-0603" value="1k1"/>
 </parts>
 <sheets>
@@
 <text x="66.04" y="88.9" size="1.778" layer="91" align="center-right">BPIO1</text>
 <text x="66.04" y="109.22" size="1.778" layer="91" align="center-right">GND</text>
+<text x="76.2" y="71.12" size="1.778" layer="91" align="center-right">TEST POINT</text>
 </plain>
 <instances>
@@
 <attribute name="VALUE" x="196.088" y="133.985" size="1.778" layer="96"/>
 </instance>
+<instance part="LED17" gate="LED" x="198.12" y="96.52" smashed="yes" rot="R90">
+<attribute name="NAME" x="198.12" y="99.06" size="1.778" layer="95" rot="R180" align="center-right"/>
+<attribute name="VALUE" x="202.692" y="102.235" size="1.778" layer="96" rot="R180"/>
+</instance>
+<instance part="SUPPLY10" gate="G$1" x="203.2" y="91.44" smashed="yes"/>
+<instance part="J2" gate="J" x="71.12" y="63.5" rot="MR0"/>
+<instance part="SUPPLY11" gate="G$1" x="76.2" y="58.42" smashed="yes"/>
+<instance part="R9" gate="R" x="190.5" y="96.52" smashed="yes">
+<attribute name="NAME" x="186.69" y="98.0186" size="1.778" layer="95" font="vector"/>
+<attribute name="VALUE" x="186.69" y="93.218" size="1.778" layer="96" font="vector"/>
+</instance>
 </instances>
 <busses>
@@
 <wire x1="73.66" y1="109.22" x2="76.2" y2="109.22" width="0.1524" layer="91"/>
 <pinref part="SUPPLY2" gate="G$1" pin="DGND"/>
+</segment>
+<segment>
+<pinref part="LED17" gate="LED" pin="C"/>
+<pinref part="SUPPLY10" gate="G$1" pin="DGND"/>
+<wire x1="203.2" y1="96.52" x2="203.2" y2="93.98" width="0.1524" layer="91"/>
+<label x="203.2" y="88.9" size="1.778" layer="95"/>
+</segment>
+<segment>
+<pinref part="J2" gate="J" pin="2"/>
+<pinref part="SUPPLY11" gate="G$1" pin="DGND"/>
+<wire x1="71.12" y1="60.96" x2="76.2" y2="60.96" width="0.1524" layer="91"/>
+<label x="76.2" y="60.96" size="1.778" layer="95"/>
 </segment>
 </net>
@@
 <label x="149.86" y="58.42" size="1.778" layer="95" align="center-left"/>
 </segment>
-</net>
+<segment>
+<pinref part="J2" gate="J" pin="1"/>
+<wire x1="71.12" y1="63.5" x2="76.2" y2="63.5" width="0.1524" layer="91"/>
+<label x="76.2" y="63.5" size="1.778" layer="95"/>
+</segment>
+<segment>
+<pinref part="R9" gate="R" pin="1"/>
+<wire x1="185.42" y1="96.52" x2="182.88" y2="96.52" width="0.1524" layer="91"/>
+<label x="182.88" y="96.52" size="1.778" layer="95" align="center-right"/>
+</segment>
+</net>
+<net name="N$9" class="0">
+<segment>
+<pinref part="LED17" gate="LED" pin="A"/>
+<pinref part="R9" gate="R" pin="2"/>
+</segment>
+</net>
