File: BPUv1b/BusPirate-ultra.v1.0b.sch (EAGLE design)
At the start: 168 parts, among them IC1 23LC1024, IC10 SN74LVC1T45DBV, IC11 SN74LVC1T45DBV, IC12 74LVC1G07DBV, IC13 SN74LVC1T45DBV, IC17 74LVC1G07DBV, IC18 SN74LVC1T45DBV, IC19 74LVC1G07DBV, IC2 23LC1024, IC20 SN74LVC1T45DBV, IC21 74LVC1G07DBV, IC22 SN74LVC1T45DBV, IC23 MCP1824_ADJ, IC24 74HCT4051, IC4 74LVC1G07DBV, IC5 74LVC1G07DBV, IC6 74LVC1G07DBV, IC7 74LVC1G07DBV, IC8 SN74LVC1T45DBV, IC9 SN74LVC1T45DBV, J1 CON_MOLEX_MALE_SMT_SH_1.25, J2 CON_HEADER_1X04, J4 CON_HEADER_1X10-RIGHT_ANGLED_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, Q1 DMMT3906W, U1 W25X40CL, U2 STM32F103ZX, U3 ICE40HX4K, U4 MCP6001, U5 74LVC245A, U7 MCP6001, U8 74HCT4066PW, U9 74HCT4066PW

Commit message: continue routing
Parts:
- removed R10, R7, R8, R9: 10K, resistor:R-EU_R0603
- added RN1: 10K, dp_devices:RNETWORK
Connections:
- removed net N$65: R51.2, R9.1
- new net N$21: R51.2, RN1D.1
- net ADC1: now also RN1C.2, RN1D.2; no longer R10.2, R9.2
- net GND: now also RN1B.1, RN1C.1; no longer R10.1, R8.1
- net MCU_ADC6: now also RN1A.2, RN1B.2; no longer R7.2, R8.2
- net VREF/VOUT: now also RN1A.1; no longer R7.1
Changed lines of the file:
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@@
 <part name="C52" library="rcl" deviceset="C-EU" device="C0603" value="0.1uF"/>
 <part name="C54" library="rcl" deviceset="C-EU" device="C0603" value="0.1uF"/>
-<part name="R9" library="resistor" deviceset="R-EU_" device="R0603" value="10K"/>
-<part name="R10" library="resistor" deviceset="R-EU_" device="R0603" value="10K"/>
 <part name="FRAME1" library="frames" deviceset="FRAME_A_L" device=""/>
 <part name="R1" library="rcl" library_urn="urn:adsk.eagle:library:334" deviceset="R-EU_" device="R0603" package3d_urn="urn:adsk.eagle:package:23555/3" value="1.5K"/>
@@
 <part name="GND7" library="dp_devices.v6" deviceset="SUPPLY_GND" device=""/>
 <part name="GND11" library="dp_devices.v6" deviceset="SUPPLY_GND" device=""/>
-<part name="GND12" library="dp_devices.v6" deviceset="SUPPLY_GND" device=""/>
 <part name="GND15" library="dp_devices.v6" deviceset="SUPPLY_GND" device=""/>
 <part name="GND16" library="dp_devices.v6" deviceset="SUPPLY_GND" device=""/>
@@
 <part name="FRAME5" library="frames" deviceset="FRAME_A_L" device=""/>
 <part name="GND64" library="dp_devices.v6" deviceset="SUPPLY_GND" device=""/>
-<part name="R7" library="resistor" deviceset="R-EU_" device="R0603" value="10K"/>
-<part name="R8" library="resistor" deviceset="R-EU_" device="R0603" value="10K"/>
 <part name="GND77" library="dp_devices.v6" deviceset="SUPPLY_GND" device=""/>
 <part name="SUPPLY4" library="supply2" deviceset="V+" device=""/>
@@
 <part name="R49" library="rcl" library_urn="urn:adsk.eagle:library:334" deviceset="R-EU_" device="R0603" package3d_urn="urn:adsk.eagle:package:23555/3" value="5K1"/>
 <part name="R52" library="rcl" library_urn="urn:adsk.eagle:library:334" deviceset="R-EU_" device="R0603" package3d_urn="urn:adsk.eagle:package:23555/3" value="5K1"/>
+<part name="RN1" library="dp_devices" deviceset="RNETWORK" device="" value="10K"/>
+<part name="GND14" library="dp_devices.v6" deviceset="SUPPLY_GND" device=""/>
 </parts>
 <sheets>
@@
 <attribute name="VALUE" x="510.54" y="332.74" size="1.778" layer="96" rot="R90"/>
 </instance>
-<instance part="R9" gate="G$1" x="411.48" y="378.46" smashed="yes" rot="MR180">
-<attribute name="NAME" x="411.48" y="375.92" size="1.778" layer="95" rot="MR180" align="center"/>
-<attribute name="VALUE" x="411.48" y="373.38" size="1.778" layer="96" rot="MR180" align="center"/>
-</instance>
-<instance part="R10" gate="G$1" x="416.56" y="373.38" smashed="yes" rot="MR90">
-<attribute name="NAME" x="421.64" y="373.38" size="1.778" layer="95" rot="MR180" align="center"/>
-<attribute name="VALUE" x="421.64" y="370.84" size="1.778" layer="96" rot="MR180" align="center"/>
-</instance>
 <instance part="FRAME1" gate="G$1" x="-2.54" y="228.6" smashed="yes"/>
 <instance part="FRAME1" gate="G$2" x="170.18" y="228.6" smashed="yes">
@@
 <instance part="GND7" gate="G$1" x="350.52" y="406.4" smashed="yes"/>
 <instance part="GND11" gate="G$1" x="330.2" y="378.46" smashed="yes"/>
-<instance part="GND12" gate="G$1" x="416.56" y="365.76" smashed="yes"/>
 <instance part="GND15" gate="G$1" x="256.54" y="284.48" smashed="yes"/>
 <instance part="GND16" gate="G$1" x="640.08" y="200.66" smashed="yes"/>
@@
 </instance>
 <instance part="GND64" gate="G$1" x="632.46" y="147.32" smashed="yes"/>
-<instance part="R7" gate="G$1" x="411.48" y="314.96" smashed="yes" rot="MR270">
-<attribute name="NAME" x="414.02" y="317.5" size="1.778" layer="95" rot="MR180" align="center-left"/>
-<attribute name="VALUE" x="414.02" y="314.96" size="1.778" layer="96" rot="MR180" align="center-left"/>
-</instance>
-<instance part="R8" gate="G$1" x="411.48" y="304.8" smashed="yes" rot="MR90">
-<attribute name="NAME" x="414.02" y="304.8" size="1.778" layer="95" rot="MR180" align="center-left"/>
-<attribute name="VALUE" x="414.02" y="302.26" size="1.778" layer="96" rot="MR180" align="center-left"/>
-</instance>
-<instance part="GND77" gate="G$1" x="411.48" y="297.18" smashed="yes"/>
+<instance part="GND77" gate="G$1" x="414.02" y="299.72" smashed="yes"/>
 <instance part="SUPPLY4" gate="1" x="330.2" y="332.74" smashed="yes"/>
 <instance part="SUPPLY5" gate="1" x="337.82" y="302.26" smashed="yes"/>
@@
 <attribute name="VALUE" x="632.46" y="170.18" size="1.778" layer="96" font="vector"/>
 </instance>
+<instance part="RN1" gate="A" x="414.02" y="317.5" rot="R270"/>
+<instance part="RN1" gate="B" x="414.02" y="307.34" smashed="yes" rot="R90">
+<attribute name="NAME" x="411.48" y="307.34" size="1.778" layer="95" rot="R270" align="center"/>
+<attribute name="VALUE" x="408.94" y="307.34" size="1.778" layer="96" rot="R270" align="center"/>
+</instance>
+<instance part="RN1" gate="C" x="416.56" y="373.38" rot="R90"/>
+<instance part="RN1" gate="D" x="411.48" y="378.46"/>
+<instance part="GND14" gate="G$1" x="416.56" y="365.76" smashed="yes"/>
 </instances>
 <busses>
@@
 </segment>
 <segment>
-<pinref part="R10" gate="G$1" pin="1"/>
-<pinref part="GND12" gate="G$1" pin="GND"/>
-</segment>
-<segment>
 <pinref part="LED3" gate="LED" pin="C"/>
 <pinref part="SUPPLY56" gate="GND" pin="GND"/>
@@
 </segment>
 <segment>
-<pinref part="R8" gate="G$1" pin="1"/>
-<pinref part="GND77" gate="G$1" pin="GND"/>
-</segment>
-<segment>
 <pinref part="R46" gate="R" pin="2"/>
 <pinref part="GND84" gate="G$1" pin="GND"/>
@@
 <junction x="635" y="170.18"/>
 </segment>
+<segment>
+<pinref part="RN1" gate="B" pin="1"/>
+<pinref part="GND77" gate="G$1" pin="GND"/>
+</segment>
+<segment>
+<pinref part="RN1" gate="C" pin="1"/>
+<pinref part="GND14" gate="G$1" pin="GND"/>
+</segment>
 </net>
 <net name="3V3" class="0">
@@
 </segment>
 <segment>
-<pinref part="R9" gate="G$1" pin="2"/>
-<pinref part="R10" gate="G$1" pin="2"/>
-<wire x1="416.56" y1="378.46" x2="419.1" y2="378.46" width="0.1524" layer="91"/>
+<pinref part="RN1" gate="C" pin="2"/>
+<pinref part="RN1" gate="D" pin="2"/>
+<wire x1="416.56" y1="378.46" x2="421.64" y2="378.46" width="0.1524" layer="91"/>
 <junction x="416.56" y="378.46"/>
-<label x="419.1" y="378.46" size="1.778" layer="95" align="center-left"/>
+<label x="421.64" y="378.46" size="1.778" layer="95"/>
 </segment>
 </net>
@@
 <pinref part="C64" gate="G$1" pin="1"/>
 <junction x="337.82" y="299.72"/>
-<pinref part="C64" gate="G$1" pin="1"/>
 </segment>
 <segment>
@@
 </segment>
 <segment>
-<pinref part="R7" gate="G$1" pin="2"/>
-<pinref part="R8" gate="G$1" pin="2"/>
-<wire x1="411.48" y1="309.88" x2="416.56" y2="309.88" width="0.1524" layer="91"/>
-<junction x="411.48" y="309.88"/>
-<label x="416.56" y="309.88" size="1.778" layer="95" align="center-left"/>
+<pinref part="RN1" gate="A" pin="2"/>
+<pinref part="RN1" gate="B" pin="2"/>
+<wire x1="414.02" y1="312.42" x2="419.1" y2="312.42" width="0.1524" layer="91"/>
+<junction x="414.02" y="312.42"/>
+<label x="419.1" y="312.42" size="1.778" layer="95"/>
 </segment>
 </net>
@@
 <junction x="398.78" y="327.66"/>
 <label x="416.56" y="327.66" size="1.778" layer="95" align="center-left"/>
-<wire x1="416.56" y1="327.66" x2="411.48" y2="327.66" width="0.1524" layer="91"/>
+<wire x1="416.56" y1="327.66" x2="414.02" y2="327.66" width="0.1524" layer="91"/>
 <pinref part="Q1" gate="B" pin="E"/>
 <pinref part="Q2" gate="Q" pin="S"/>
-<pinref part="R7" gate="G$1" pin="1"/>
+<wire x1="414.02" y1="327.66" x2="411.48" y2="327.66" width="0.1524" layer="91"/>
 <wire x1="411.48" y1="327.66" x2="398.78" y2="327.66" width="0.1524" layer="91"/>
-<wire x1="411.48" y1="320.04" x2="411.48" y2="327.66" width="0.1524" layer="91"/>
-<junction x="411.48" y="327.66"/>
+<pinref part="RN1" gate="A" pin="1"/>
+<wire x1="414.02" y1="322.58" x2="414.02" y2="327.66" width="0.1524" layer="91"/>
+<junction x="414.02" y="327.66"/>
 </segment>
 <segment>
@@
 </segment>
 </net>
-<net name="N$65" class="0">
-<segment>
-<pinref part="R51" gate="G$1" pin="2"/>
-<pinref part="R9" gate="G$1" pin="1"/>
-</segment>
-</net>
 <net name="BPIO0" class="0">
 <segment>
@@
 </segment>
 </net>
+<net name="N$21" class="0">
+<segment>
+<pinref part="R51" gate="G$1" pin="2"/>
+<pinref part="RN1" gate="D" pin="1"/>
+</segment>
+</net>

Commit message: continue routing
Parts:
- R6: device dp_devices:RESISTOR-0603 -> rcl:R-EU_R0603
Connections:
- net FPGA_PROG_CS: now also R6.2; no longer R6.1
- net GND: now also R6.1; no longer R6.2
Other:
- moved on the sheet: R6
Changed lines of the file:
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@@
 <part name="P+6" library="supply1" library_urn="urn:adsk.eagle:library:371" deviceset="VCC" device=""/>
 <part name="P+11" library="supply1" library_urn="urn:adsk.eagle:library:371" deviceset="VCC" device=""/>
-<part name="R6" library="dp_devices" deviceset="RESISTOR" device="-0603" value="10K"/>
 <part name="R16" library="rcl" library_urn="urn:adsk.eagle:library:334" deviceset="R-EU_" device="R0603" package3d_urn="urn:adsk.eagle:package:23555/3" value="10K"/>
 <part name="R15" library="rcl" library_urn="urn:adsk.eagle:library:334" deviceset="R-EU_" device="R0603" package3d_urn="urn:adsk.eagle:package:23555/3" value="10K"/>
@@
 <part name="RN1" library="dp_devices" deviceset="RNETWORK" device="" value="10K"/>
 <part name="GND14" library="dp_devices.v6" deviceset="SUPPLY_GND" device=""/>
+<part name="R6" library="rcl" library_urn="urn:adsk.eagle:library:334" deviceset="R-EU_" device="R0603" package3d_urn="urn:adsk.eagle:package:23555/3" value="10K"/>
 </parts>
 <sheets>
@@
 <instance part="P+6" gate="VCC" x="502.92" y="299.72" smashed="yes"/>
 <instance part="P+11" gate="VCC" x="96.52" y="205.74" smashed="yes"/>
-<instance part="R6" gate="G$1" x="337.82" y="15.24" smashed="yes" rot="R270">
-<attribute name="NAME" x="330.2" y="15.24" size="1.778" layer="95"/>
-<attribute name="VALUE" x="330.2" y="12.7" size="1.778" layer="96"/>
-</instance>
 <instance part="R16" gate="G$1" x="533.4" y="78.74" smashed="yes" rot="R90">
 <attribute name="NAME" x="535.94" y="78.74" size="1.778" layer="95"/>
@@
 <instance part="RN1" gate="D" x="411.48" y="378.46"/>
 <instance part="GND14" gate="G$1" x="416.56" y="365.76" smashed="yes"/>
+<instance part="R6" gate="G$1" x="337.82" y="15.24" smashed="yes" rot="R90">
+<attribute name="NAME" x="340.36" y="15.24" size="1.778" layer="95"/>
+<attribute name="VALUE" x="340.36" y="12.7" size="1.778" layer="96"/>
+</instance>
 </instances>
 <busses>
@@
 <wire x1="88.9" y1="203.2" x2="86.36" y2="203.2" width="0.1524" layer="91"/>
 <junction x="88.9" y="203.2"/>
-</segment>
-<segment>
-<pinref part="R6" gate="G$1" pin="2"/>
-<pinref part="GND67" gate="G$1" pin="GND"/>
 </segment>
 <segment>
@@
 <pinref part="GND14" gate="G$1" pin="GND"/>
 </segment>
+<segment>
+<pinref part="GND67" gate="G$1" pin="GND"/>
+<pinref part="R6" gate="G$1" pin="1"/>
+</segment>
 </net>
 <net name="3V3" class="0">
@@
 <wire x1="340.36" y1="20.32" x2="337.82" y2="20.32" width="0.1524" layer="91"/>
 <label x="335.28" y="20.32" size="1.778" layer="95" align="center-right"/>
-<pinref part="R6" gate="G$1" pin="1"/>
 <wire x1="337.82" y1="20.32" x2="335.28" y2="20.32" width="0.1524" layer="91"/>
+<pinref part="R6" gate="G$1" pin="2"/>
 <junction x="337.82" y="20.32"/>
 </segment>

Commit message: board routing done, add usbc bottom PTH chassis mount library
Parts:
- removed C65: 0.1uF, rcl:C-EUC0603
- removed IC13, IC18, IC20, IC22: SN74LVC1T45DBV, dp_devices.v6:IC_BUFF_SN74LVC1T45DBV-EXTENDED
- removed IC17, IC19, IC21: 74LVC1G07DBV, dp_devices.v6:IC_BUFF_74LVC1G07-EXTENDED
- removed IC23: MCP1824_ADJ, dp_devices.v6:IC_MCP1824_ADJ
- removed IC24: 74HCT4051, dp_devices.v6:IC_74HCT4051
- removed J4: CON_HEADER_1X10-RIGHT_ANGLED_PTH_SHROUDED, dp_devices.v6:CON_HEADER_1X10-RIGHT_ANGLED_PTH_SHROUDED
- removed R50, R51: (no value), resistor:R-EU_R0603
- removed R52: 5K1, rcl:R-EU_R0603
- removed R53: 0R, dp_devices.v6:RESISTOR-0603
- removed RN4: 2K, dp_devices:RNETWORK
- removed U$3: USB-C-12, usbc:USB-C-12
- added C62: 0.1uF, rcl:C-EUC0603
- added CON1: USB-C-12, usbc:USB-C-12
- added IC3: SN74LVC1T45DBV, dp_devices.v6:IC_BUFF_SN74LVC1T45DBV-EXTENDED
- added J3: CON_MOLEX_MALE_SMT_SH_1.25, dp_devices.v6:CON_MOLEX_MALE_SMT_SH_1.25
- added R10, R8: 1M, resistor:R-EU_R0402
- added R7, R9: 100K, resistor:R-EU_R0402
- added RN2: 2K, dp_devices:RNETWORK
- added U10, U11: 74HCT4066PW, dp_devices.v6:IC_74HCT4066PW
- added U12: W25X40CL, dp_devices.v6:IC_MEM_W25X40CL
- added U13: 74LVC245A, dp_devices.v6:IC_BUFF_74LVC245A-TSSOP20
- added U14: MCP6001, dp_devices.v6:IC_OP-AMP_MCP6001
- added U15: MCP6001, dp_devices.v6:IC_MCP6001
- added U16: ICE40HX4K, dp_devices.v6:IC_FPGA_ICE40HX4K
- added U6: 74LVC1G07DBV, dp_devices.v6:IC_BUFF_74LVC1G07-EXTENDED
- C1: value 10uF -> 0.1uF; device rcl:CPOL-EUSMCA -> rcl:C-EUC0402
- C10: device dp_devices.v6:CAPACITOR_NPOL-0402 -> resistor:C-EUC0402
- C11, C12, C13, C14, C15, C2, C3, C4, C6, C7, C8, C9: device rcl:C-EUC0603 -> resistor:C-EUC0402
- C16: value 22pF -> 0.1uF; device rcl:C-EUC0603 -> resistor:C-EUC0402
- C17: value 1uF -> 0.1uF; device rcl:CPOL-EUSMCA -> rcl:C-EUC0603
- C19: value 0.1uF -> 1uF; device rcl:C-EUC0603 -> rcl:CPOL-EUSMCA
- C20: value 0.1uF -> 22pF; device dp_devices.v6:CAPACITOR_NPOL-0402 -> rcl:C-EUC0603
- C23: value 0.1uF -> 10uF; device rcl:C-EUC0603 -> dp_devices.v6:CAPACITOR_NPOL-0603
- C24: value 0.1uF -> (none)
- C27: device dp_devices.v6:CAPACITOR_NPOL-0402 -> rcl:C-EUC0603
- C28: value 0.1uF -> 1uf
- C29: value 0.1uF -> 1uF; device rcl:C-EUC0603 -> dp_devices.v6:CAPACITOR_NPOL-0603
- C32: device rcl:C-EUC0603 -> dp_devices.v6:CAPACITOR_NPOL-0402
- C36: value 1uf -> 0.1uF; device rcl:C-EUC0603 -> dp_devices.v6:CAPACITOR_NPOL-0402
- C38: value 1uf -> 1uF
- C39: value 0.1uF -> 1uf; device rcl:C-EUC0402 -> rcl:C-EUC0603
- C40, C41, C42, C43, C46, C47, C48, C49, C55, C56, C57, C58, C60: device resistor:C-EUC0402 -> rcl:C-EUC0603
- C45: device rcl:C-EUC0402 -> rcl:C-EUC0603
- C5: device rcl:C-EUC0603 -> rcl:C-EUC0402
- C51: value 1uF -> 0.1uF
- C53: value (none) -> 0.1uF
- C59: device resistor:C-EUC0402 -> dp_devices.v6:CAPACITOR_NPOL-0402
- C61: value 1uF -> 0.1uF; device dp_devices.v6:CAPACITOR_NPOL-0603 -> rcl:C-EUC0603
- C63: value 10uF -> 0.1uF; device dp_devices.v6:CAPACITOR_NPOL-0603 -> rcl:C-EUC0603
- C64: value 0.1uF -> 10uF; device rcl:C-EUC0603 -> rcl:CPOL-EUSMCA
- IC1, IC2: value 23LC1024 -> SN74LVC1T45DBV; device dp_devices:IC_MEM_23LC1024 -> dp_devices.v6:IC_BUFF_SN74LVC1T45DBV-EXTENDED
- IC10, IC9: value SN74LVC1T45DBV -> 23LC1024; device dp_devices.v6:IC_BUFF_SN74LVC1T45DBV-EXTENDED -> dp_devices:IC_MEM_23LC1024
- IC11: value SN74LVC1T45DBV -> 74HCT4051; device dp_devices.v6:IC_BUFF_SN74LVC1T45DBV-EXTENDED -> dp_devices.v6:IC_74HCT4051
- IC12: value 74LVC1G07DBV -> MCP1824_ADJ; device dp_devices.v6:IC_BUFF_74LVC1G07-EXTENDED -> dp_devices.v6:IC_MCP1824_ADJ
- IC4, IC5, IC6, IC7: value 74LVC1G07DBV -> SN74LVC1T45DBV; device dp_devices.v6:IC_BUFF_74LVC1G07-EXTENDED -> dp_devices.v6:IC_BUFF_SN74LVC1T45DBV-EXTENDED
- J1: value CON_MOLEX_MALE_SMT_SH_1.25 -> CON_HEADER_1X04; device dp_devices.v6:CON_MOLEX_MALE_SMT_SH_1.25 -> dp_devices.v6:CON_HEADER_1X04
- J2: value CON_HEADER_1X04 -> CON_HEADER_1X10-RIGHT_ANGLED_PTH_SHROUDED; device dp_devices.v6:CON_HEADER_1X04 -> dp_devices.v6:CON_HEADER_1X10-RIGHT_ANGLED_PTH_SHROUDED
- R1: value 1.5K -> 100K; device rcl:R-EU_R0603 -> resistor:R-EU_R0402
- R11: value 10K -> 100K; device resistor:R-EU_R0603 -> resistor:R-EU_R0402
- R12: value 10K -> 1M; device resistor:R-EU_R0603 -> resistor:R-EU_R0402
- R13, R14, R17: value 1K1 -> 100K; device dp_devices:RESISTOR-0603 -> resistor:R-EU_R0402
- R15, R16: value 10K -> 100K; device rcl:R-EU_R0603 -> resistor:R-EU_R0402
- R18: value 1K1 -> 1M; device dp_devices:RESISTOR-0603 -> resistor:R-EU_R0402
- R2, R3: value 22R -> 100K; device rcl:R-EU_R0603 -> resistor:R-EU_R0402
- R20, R22: value 100K -> 1M
- R25, R27: value 1M -> 10K; device resistor:R-EU_R0402 -> dp_devices.v6:RESISTOR-0603
- R26: value 1M -> (none); device resistor:R-EU_R0402 -> rcl:R-EU_R0603
- R28: value 100K -> 0R; device resistor:R-EU_R0402 -> dp_devices.v6:RESISTOR-0603
- R29, R37, R38: value 100K -> 10K; device resistor:R-EU_R0402 -> rcl:R-EU_R0603
- R30: value 100K -> 78.7K; device resistor:R-EU_R0402 -> dp_devices.v6:RESISTOR-0603
- R31: value 1M -> 100K; device resistor:R-EU_R0402 -> dp_devices.v6:RESISTOR-0603
- R32: value 100K -> 50K; device resistor:R-EU_R0402 -> dp_devices.v6:RESISTOR-0603
- R33: value 100K -> (none); device resistor:R-EU_R0402 -> resistor:R-EU_R0603
- R34, R35: value 100K -> (none); device resistor:R-EU_R0402 -> dp_devices.v6:RESISTOR-0603
- R36: value 1M -> (none); device resistor:R-EU_R0402 -> resistor:R-EU_R0603
- R39: value 1M -> 10K; device resistor:R-EU_R0402 -> resistor:R-EU_R0603
- R4, R5: value 10K -> 100K; device dp_devices.v6:RESISTOR-0603 -> resistor:R-EU_R0402
- R40: value 100K -> 10K; device resistor:R-EU_R0402 -> resistor:R-EU_R0603
- R41: value 100K -> 1.5K; device resistor:R-EU_R0402 -> rcl:R-EU_R0603
- R42: value 1M -> 22R; device resistor:R-EU_R0402 -> rcl:R-EU_R0603
- R43: value (none) -> 22R; device dp_devices.v6:RESISTOR-0603 -> rcl:R-EU_R0603
- R44: value (none) -> 5K1; device dp_devices.v6:RESISTOR-0603 -> rcl:R-EU_R0603
- R45: value 100K -> 5K1; device dp_devices.v6:RESISTOR-0603 -> rcl:R-EU_R0603
- R46: value 50K -> 1K1; device dp_devices.v6:RESISTOR-0603 -> dp_devices:RESISTOR-0603
- R47: value 78.7K -> 1K1; device dp_devices.v6:RESISTOR-0603 -> dp_devices:RESISTOR-0603
- R48: value (none) -> 1K1; device rcl:R-EU_R0603 -> dp_devices:RESISTOR-0603
- R49: value 5K1 -> 1K1; device rcl:R-EU_R0603 -> dp_devices:RESISTOR-0603
- R6: value 10K -> 1M; device rcl:R-EU_R0603 -> resistor:R-EU_R0402
- RN1: value 10K -> 2K
- RN3: value 2K -> 10K
- U1: value W25X40CL -> 74LVC1G07DBV; device dp_devices.v6:IC_MEM_W25X40CL -> dp_devices.v6:IC_BUFF_74LVC1G07-EXTENDED
- U2: value STM32F103ZX -> 74LVC1G07DBV; device dp_devices.v6:IC_UC_STM32F103ZX -> dp_devices.v6:IC_BUFF_74LVC1G07-EXTENDED
- U3: value ICE40HX4K -> 74LVC1G07DBV; device dp_devices.v6:IC_FPGA_ICE40HX4K -> dp_devices.v6:IC_BUFF_74LVC1G07-EXTENDED
- U4: value MCP6001 -> 74LVC1G07DBV; device dp_devices.v6:IC_OP-AMP_MCP6001 -> dp_devices.v6:IC_BUFF_74LVC1G07-EXTENDED
- U5: value 74LVC245A -> STM32F103ZX; device dp_devices.v6:IC_BUFF_74LVC245A-TSSOP20 -> dp_devices.v6:IC_UC_STM32F103ZX
- U7: value MCP6001 -> 74LVC1G07DBV; device dp_devices.v6:IC_MCP6001 -> dp_devices.v6:IC_BUFF_74LVC1G07-EXTENDED
- U8, U9: value 74HCT4066PW -> 74LVC1G07DBV; device dp_devices.v6:IC_74HCT4066PW -> dp_devices.v6:IC_BUFF_74LVC1G07-EXTENDED
- renumbered VR3 to VR2
Connections:
- net 1V2: now also C36.1, C39.1, C43.2, C54.2, C55.2, U16BANK0.VCC@0, U16BANK0.VCCPLL1, U16BANK1.VCC@0, U16BANK2.VCC@0, U16BANK2.VCCPLL0, U16BANK3.VCC@0; no longer C23.2, C26.2, C27.1, C33.2, C38.1, U3BANK0.VCC@0, U3BANK0.VCCPLL1, U3BANK1.VCC@0, U3BANK2.VCC@0, U3BANK2.VCCPLL0, U3BANK3.VCC@0
- net 3V3: now also C1.1, C11.1, C12.1, C17.2, C19.+, C2.1, C28.1, C3.1, C32.1, C33.2, C4.1, C42.2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; no longer C11.2, C12.2, C13.2, C15.2, C17.+, C19.2, C2.2, C20.1, C24.2, C28.2, C29.2, C3.2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
- net ADC1: now also RN3C.2, RN3D.2, U5U.ADC12_IN9/TIM3_CH4('00'OR'10')/TIM8_CH3N/TIM1_CH3N('01')/PB1; no longer RN1C.2, RN1D.2, U2U.ADC12_IN9/TIM3_CH4('00'OR'10')/TIM8_CH3N/TIM1_CH3N('01')/PB1
- net ADC_MUX_EN: now also IC11.!E, U16BANK1.IOR_146; no longer IC24.!E, U3BANK1.IOR_146
- net ADC_MUX_S0: now also IC11.S0, U16BANK1.GBIN3/IOR_140; no longer IC24.S0, U3BANK1.GBIN3/IOR_140
- net ADC_MUX_S1: now also IC11.S1, U16BANK1.GBIN2/IOR_141; no longer IC24.S1, U3BANK1.GBIN2/IOR_141
- net ADC_MUX_S2: now also IC11.S2, U16BANK1.IOR_144; no longer IC24.S2, U3BANK1.IOR_144
- net BPIO0: now also IC1.B, IC11.Y0, J2.1, R6.2, RN1A.1, U13G$1.B0, U1G.O; no longer IC24.Y0, IC4G.O, IC8.B, J4.1, R24.2, RN4A.1, U5G$1.B0
- net BPIO1: now also IC11.Y1, IC2.B, J2.2, R8.2, RN1B.1, U13G$1.B1, U2G.O; no longer IC24.Y1, IC5G.O, IC9.B, J4.2, R25.2, RN4B.1, U5G$1.B1
- net BPIO2: now also IC11.Y2, IC3.B, J2.3, R10.2, RN1C.1, U13G$1.B2, U3G.O; no longer IC10.B, IC24.Y2, IC6G.O, J4.3, R26.2, RN4C.1, U5G$1.B2
- net BPIO3: now also IC11.Y3, IC4.B, J2.4, R12.2, RN1D.1, U13G$1.B3, U4G.O; no longer IC12G.O, IC13.B, IC24.Y3, J4.4, R31.2, RN4D.1, U5G$1.B3
- net BPIO4: now also IC11.Y4, IC5.B, J2.5, R18.2, RN2D.2, U13G$1.B4, U6G.O; no longer IC11.B, IC24.Y4, IC7G.O, J4.5, R27.2, RN3D.2, U5G$1.B4
- net BPIO5: now also IC11.Y5, IC6.B, J2.6, R20.2, RN2C.2, U13G$1.B5, U7G.O; no longer IC17G.O, IC18.B, IC24.Y5, J4.6, R36.2, RN3C.2, U5G$1.B5
- net BPIO6: now also IC11.Y6, IC7.B, J2.7, R22.2, RN2B.2, U13G$1.B6, U8G.O; no longer IC19G.O, IC20.B, IC24.Y6, J4.7, R39.2, RN3B.2, U5G$1.B6
- net BPIO7: now also IC11.Y7, IC8.B, J2.8, R24.2, RN2A.2, U13G$1.B7, U9G.O; no longer IC21G.O, IC22.B, IC24.Y7, J4.8, R42.2, RN3A.2, U5G$1.B7
- net BUFDIR0: now also IC1.DIR, R5.2, U16BANK1.IOR_167; no longer IC8.DIR, R28.2, U3BANK1.IOR_167
- net BUFDIR1: now also IC2.DIR, R7.2, U16BANK0.IOT_170; no longer IC9.DIR, R29.2, U3BANK0.IOT_170
- net BUFDIR2: now also IC3.DIR, R9.2, U16BANK1.IOR_152; no longer IC10.DIR, R30.2, U3BANK1.IOR_152
- net BUFDIR3: now also IC4.DIR, R11.2, U16BANK1.IOR_164; no longer IC13.DIR, R33.2, U3BANK1.IOR_164
- net BUFDIR4: now also IC5.DIR, R17.2, U16BANK1.IOR_115; no longer IC11.DIR, R32.2, U3BANK1.IOR_115
- net BUFDIR5: now also IC6.DIR, R19.2, U16BANK1.IOR_111; no longer IC18.DIR, R35.2, U3BANK1.IOR_111
- net BUFDIR6: now also IC7.DIR, R21.2, U16BANK2.CBSEL1/IOB_104; no longer IC20.DIR, R38.2, U3BANK2.CBSEL1/IOB_104
- net BUFDIR7: now also IC8.DIR, R23.2, U16BANK2.IOB_96; no longer IC22.DIR, R41.2, U3BANK2.IOB_96
- net BUFIO0: now also IC1.A, U16BANK1.IOR_166; no longer IC8.A, U3BANK1.IOR_166
- net BUFIO1: now also IC2.A, U16BANK0.IOT_169; no longer IC9.A, U3BANK0.IOT_169
- net BUFIO2: now also IC3.A, U16BANK1.IOR_148; no longer IC10.A, U3BANK1.IOR_148
- net BUFIO3: now also IC4.A, U16BANK1.IOR_161; no longer IC13.A, U3BANK1.IOR_161
- net BUFIO4: now also IC5.A, U16BANK1.IOR_114; no longer IC11.A, U3BANK1.IOR_114
- net BUFIO5: now also IC6.A, U16BANK1.IOR_110; no longer IC18.A, U3BANK1.IOR_110
- net BUFIO6: now also IC7.A, U16BANK2.CBSEL0/IOB_103; no longer IC20.A, U3BANK2.CBSEL0/IOB_103
- net BUFIO7: now also IC8.A, U16BANK2.IOB_95; no longer IC22.A, U3BANK2.IOB_95
- net BUFOD0: now also R1.1, U16BANK1.IOR_165, U1G.I; no longer IC4G.I, R19.1, U3BANK1.IOR_165
- net BUFOD1: now also R2.1, U16BANK0.IOT_168, U2G.I; no longer IC5G.I, R20.1, U3BANK0.IOT_168
- net BUFOD2: now also R3.1, U16BANK1.IOR_147, U3G.I; no longer IC6G.I, R21.1, U3BANK1.IOR_147
- net BUFOD3: now also R4.1, U16BANK1.IOR_160, U4G.I; no longer IC12G.I, R23.1, U3BANK1.IOR_160
- net BUFOD4: now also R13.1, U16BANK1.IOR_112, U6G.I; no longer IC7G.I, R22.1, U3BANK1.IOR_112
- net BUFOD5: now also R14.1, U16BANK1.IOR_109, U7G.I; no longer IC17G.I, R34.1, U3BANK1.IOR_109
- net BUFOD6: now also R15.1, U16BANK2.IOB_102, U8G.I; no longer IC19G.I, R37.1, U3BANK2.IOB_102
- net BUFOD7: now also R16.1, U16BANK2.IOB_94, U9G.I; no longer IC21G.I, R40.1, U3BANK2.IOB_94
- net D+: now also CON1.DP1, CON1.DP2, R41.1, R42.2; no longer R1.1, R3.2, U$3.DP1, U$3.DP2
- net D-: now also CON1.DN1, CON1.DN2, R43.2; no longer R2.2, U$3.DN1, U$3.DN2
- net DISPLAY_AUX1: now also J3.5, U5U.ADC12_IN14/PC4; no longer J1.5, U2U.ADC12_IN14/PC4
- net DISPLAY_AUX2: now also J3.4, U5U.ADC12_IN15/PC5; no longer J1.4, U2U.ADC12_IN15/PC5
- net DISPLAY_CS: now also J3.1, U5U.FSMC_A6/FT/PF12; no longer J1.1, U2U.FSMC_A6/FT/PF12
- net DISPLAY_D/P: now also J3.2, U5U.FSMC_NIOS16/FT/PF11; no longer J1.2, U2U.FSMC_NIOS16/FT/PF11
- net DISPLAY_PWM: now also J3.3, U5U.ADC12_IN8/TIM3_CH3('00'OR'10')/TIM8_CH2N/TIM1_CH2N('01')/PB0; no longer J1.3, U2U.ADC12_IN8/TIM3_CH3('00'OR'10')/TIM8_CH2N/TIM1_CH2N('01')/PB0
- net DISPLAY_SPI_CLOCK: now also J3.8, U5U.PA5/SPI1_SCK('0')/ADC12_IN5; no longer J1.8, U2U.PA5/SPI1_SCK('0')/ADC12_IN5
- net DISPLAY_SPI_MISO: now also J3.7, U5U.PA6/SPI1_MISO('0')/TIM8_BKIN/ADC12_IN6/TIM3_CH1('00')/TIM1_BKIN('01'); no longer J1.7, U2U.PA6/SPI1_MISO('0')/TIM8_BKIN/ADC12_IN6/TIM3_CH1('00')/TIM1_BKIN('01')
- net DISPLAY_SPI_MOSI: now also J3.6, U5U.PA7/SPI1_MOSI('0')/TIM8_CH1N/ADC12_IN7/TIM3_CH2('00')/TIM1_CH1N('01'); no longer J1.6, U2U.PA7/SPI1_MOSI('0')/TIM8_CH1N/ADC12_IN7/TIM3_CH2('00')/TIM1_CH1N('01')
- net FLASH_CS: now also U12.!CS, U5U.PG15/FT; no longer U1.!CS, U2U.PG15/FT
- net FLASH_MISO: now also U12.SO, U5U.SPI3_MISO('0')/TIM3_CH1('10')/SPI1_MISO('1')/NJTRST/FT/PB4; no longer U1.SO, U2U.SPI3_MISO('0')/TIM3_CH1('10')/SPI1_MISO('1')/NJTRST/FT/PB4
- net FLASH_MOSI: now also U12.SI, U5U.I2C1_SMBA/SPI3_MOSI('0')/TIM3_CH2('10')/SPI1_MOSI('1')/PB5; no longer U1.SI, U2U.I2C1_SMBA/SPI3_MOSI('0')/TIM3_CH2('10')/SPI1_MOSI('1')/PB5
- net FLASH_SCK: now also U12.SCK, U5U.SPI3_SCK('0')/TIM2_CH2('01')/SPI1_SCK('1')/JTDO/FT//PB3; no longer U1.SCK, U2U.SPI3_SCK('0')/TIM2_CH2('01')/SPI1_SCK('1')/JTDO/FT//PB3
- net FPGA_CDONE: now also R37.1, U16BANK2.CDONE, U5U.I2C2_SCL/USART3_TX('00')/TIM2_CH3('10'OR'11')/FT/PB10; no longer R15.1, U2U.I2C2_SCL/USART3_TX('00')/TIM2_CH3('10'OR'11')/FT/PB10, U3BANK2.CDONE
- net FPGA_CRESET: now also R38.1, U16BANK2.CRESET_B, U5U.I2C2_SDA/USART3_RX('00')/TIM2_CH4('10'OR'11')/FT/PB11; no longer R16.1, U2U.I2C2_SDA/USART3_RX('00')/TIM2_CH4('10'OR'11')/FT/PB11, U3BANK2.CRESET_B
- net FPGA_PROG_CLOCK: now also U16SPI.IOB_107/SCK, U5U.SPI2_SCK/USART3_CTS('00'OR'01')/TIM1_CH1N('00')/FT/PB13; no longer U2U.SPI2_SCK/USART3_CTS('00'OR'01')/TIM1_CH1N('00')/FT/PB13, U3SPI.IOB_107/SCK
- net FPGA_PROG_CS: now also R29.2, U16SPI.IOB_108/SS, U5U.SPI2_NSS/I2C2_SMBA/USART3_CK(00)/TIM1_BKIN('00')/FT/PB12; no longer R6.2, U2U.SPI2_NSS/I2C2_SMBA/USART3_CK(00)/TIM1_BKIN('00')/FT/PB12, U3SPI.IOB_108/SS
- net FPGA_PROG_MISO: now also U16SPI.IOB_105/SDO, U5U.SPI2_MISO/USART3_RTS('00'OR'01')/TIM1_CH2N('00')/FT/PB14; no longer U2U.SPI2_MISO/USART3_RTS('00'OR'01')/TIM1_CH2N('00')/FT/PB14, U3SPI.IOB_105/SDO
- net FPGA_PROG_MOSI: now also U16SPI.IOB_106/SDI, U5U.SPI2_MOSI/TIM1_CH3N('00')/FT/PB15; no longer U2U.SPI2_MOSI/TIM1_CH3N('00')/FT/PB15, U3SPI.IOB_106/SDI
- net FSMC_A0: now also U16BANK3.IOL_3A, U5U.FSMC_A0/FT/PF0; no longer U2U.FSMC_A0/FT/PF0, U3BANK3.IOL_3A
- net FSMC_A1: now also U16BANK3.IOL_3B, U5U.FSMC_A1/FT/PF1; no longer U2U.FSMC_A1/FT/PF1, U3BANK3.IOL_3B
- net FSMC_A2: now also U16BANK3.IOL_4A, U5U.FSMC_A2/FT/PF2; no longer U2U.FSMC_A2/FT/PF2, U3BANK3.IOL_4A
- net FSMC_A3: now also U16BANK3.IOL_4B, U5U.FSMC_A3/FT/PF3; no longer U2U.FSMC_A3/FT/PF3, U3BANK3.IOL_4B
- net FSMC_A4: now also U16BANK3.IOL_5A, U5U.FSMC_A4/FT/PF4; no longer U2U.FSMC_A4/FT/PF4, U3BANK3.IOL_5A
- net FSMC_A5: now also U16BANK3.IOL_5B, U5U.FSMC_A5/FT/PF5; no longer U2U.FSMC_A5/FT/PF5, U3BANK3.IOL_5B
- net FSMC_D0: now also U16BANK3.IOL_17B, U5U.PD14/FT/FSMC_D0/TIM4_CH3('1'); no longer U2U.PD14/FT/FSMC_D0/TIM4_CH3('1'), U3BANK3.IOL_17B
- net FSMC_D1: now also U16BANK3.IOL_17A, U5U.PD15/FT/FSMC_D1/TIM4_CH4('1'); no longer U2U.PD15/FT/FSMC_D1/TIM4_CH4('1'), U3BANK3.IOL_17A
- net FSMC_D10: now also U16BANK3.IOL_18B, U5U.PE13/FT/FSMC_D10/TIM1_CH3('11'); no longer U2U.PE13/FT/FSMC_D10/TIM1_CH3('11'), U3BANK3.IOL_18B
- net FSMC_D11: now also U16BANK3.IOL_23A, U5U.PE14/FT/FSMC_D11/TIM1_CH4('11'); no longer U2U.PE14/FT/FSMC_D11/TIM1_CH4('11'), U3BANK3.IOL_23A
- net FSMC_D12: now also U16BANK3.IOL_23B, U5U.PE15/FT/FSMC_D12/TIM1_BKIN('11'); no longer U2U.PE15/FT/FSMC_D12/TIM1_BKIN('11'), U3BANK3.IOL_23B
- net FSMC_D13: now also U16BANK3.IOL_25A, U5U.PD8/FT/FSMC_D13/USART3_TX('11'); no longer U2U.PD8/FT/FSMC_D13/USART3_TX('11'), U3BANK3.IOL_25A
- net FSMC_D14: now also U16BANK3.IOL_24B, U5U.PD9/FT/FSMC_D14/USART3_RX('11'); no longer U2U.PD9/FT/FSMC_D14/USART3_RX('11'), U3BANK3.IOL_24B
- net FSMC_D15: now also U16BANK3.IOL_24A, U5U.PD10/FT/FSMC_D15/USART3_CK('11'); no longer U2U.PD10/FT/FSMC_D15/USART3_CK('11'), U3BANK3.IOL_24A
- net FSMC_D2: now also U16BANK3.IOL_2A, U5U.PD0/FT/FSMC_D2; no longer U2U.PD0/FT/FSMC_D2, U3BANK3.IOL_2A
- net FSMC_D3: now also U16BANK3.IOL_2B, U5U.PD1/FT/FSMC_D3; no longer U2U.PD1/FT/FSMC_D3, U3BANK3.IOL_2B
- net FSMC_D4: now also U16BANK3.IOL_10A, U5U.PE7/FT/FSMC_D4/TIM1_ETR('11'); no longer U2U.PE7/FT/FSMC_D4/TIM1_ETR('11'), U3BANK3.IOL_10A
- net FSMC_D5: now also U16BANK3.IOL_10B, U5U.PE8/FT/FSMC_D5/TIM1_CH1N('11'); no longer U2U.PE8/FT/FSMC_D5/TIM1_CH1N('11'), U3BANK3.IOL_10B
- net FSMC_D6: now also U16BANK3.IOL_12A, U5U.PE9/FT/FSMC_D6/TIM1_CH1('11'); no longer U2U.PE9/FT/FSMC_D6/TIM1_CH1('11'), U3BANK3.IOL_12A
- net FSMC_D7: now also U16BANK3.IOL_12B, U5U.PE10/FT/FSMC_D7/TIM1_CH2N('11'); no longer U2U.PE10/FT/FSMC_D7/TIM1_CH2N('11'), U3BANK3.IOL_12B
- net FSMC_D8: now also U16BANK3.IOL_13A, U5U.PE11/FT/FSMC_D8/TIM1_CH2('11'); no longer U2U.PE11/FT/FSMC_D8/TIM1_CH2('11'), U3BANK3.IOL_13A
- net FSMC_D9: now also U16BANK3.IOL_18A, U5U.PE12/FT/FSMC_D9/TIM1_CH3N('11'); no longer U2U.PE12/FT/FSMC_D9/TIM1_CH3N('11'), U3BANK3.IOL_18A
- net FSMC_NE3_CE: now also U16BANK3.IOL_14B, U5U.PG10/FT/FSMC_NCE4_1/FSMC_NE3; no longer U2U.PG10/FT/FSMC_NCE4_1/FSMC_NE3, U3BANK3.IOL_14B
- net FSMC_NOE_OE: now also U16BANK3.IOL_8A, U5U.PD4/FT/FSMC_NOE/USART2_RTS(1); no longer U2U.PD4/FT/FSMC_NOE/USART2_RTS(1), U3BANK3.IOL_8A
- net FSMC_NWE_WE: now also U16BANK3.IOL_8B, U5U.PD5/FT/FSMC_NWE/USART2_TX('1'); no longer U2U.PD5/FT/FSMC_NWE/USART2_TX('1'), U3BANK3.IOL_8B
- net GND: now also C1.2, C11.2, C12.2, C14.1, C17.1, C19.-, C2.2, C20.1, C23.2, C24.2, C26.2, C28.2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; no longer C1.-, C11.1, C12.1, C14.2, C17.-, C19.1, C2.1, C20.2, C23.1, C24.1, C26.1, C28.1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
- net LAT0: now also U13G$1.A0, U16BANK1.IOR_139; no longer U3BANK1.IOR_139, U5G$1.A0
- net LAT1: now also U13G$1.A1, U16BANK1.IOR_138; no longer U3BANK1.IOR_138, U5G$1.A1
- net LAT2: now also U13G$1.A2, U16BANK1.IOR_137; no longer U3BANK1.IOR_137, U5G$1.A2
- net LAT3: now also U13G$1.A3, U16BANK1.IOR_136; no longer U3BANK1.IOR_136, U5G$1.A3
- net LAT4: now also U13G$1.A4, U16BANK1.IOR_128; no longer U3BANK1.IOR_128, U5G$1.A4
- net LAT5: now also U13G$1.A5, U16BANK1.IOR_120; no longer U3BANK1.IOR_120, U5G$1.A5
- net LAT6: now also U13G$1.A6, U16BANK1.IOR_119; no longer U3BANK1.IOR_119, U5G$1.A6
- net LAT7: now also U13G$1.A7, U16BANK1.IOR_118; no longer U3BANK1.IOR_118, U5G$1.A7
- net LD1: now also R47.2, U5U.PA15/FT/JTDI/SPI3_NSS('0')/TIM2_CH1_ETR('11')/SPI1_NSS('1'); no longer R14.2, U2U.PA15/FT/JTDI/SPI3_NSS('0')/TIM2_CH1_ETR('11')/SPI1_NSS('1')
- net MCU_ADC5: now also R39.2, R40.2, U5U.PA3/USART2_RX('0')/TIM5_CH4/ADC123_IN3/TIM2_CH4('00'OR'01'); no longer R11.2, R12.2, U2U.PA3/USART2_RX('0')/TIM5_CH4/ADC123_IN3/TIM2_CH4('00'OR'01')
- net MCU_ADC6: now also RN3A.2, RN3B.2, U5U.PA2/USART2_TX('0')/TIM5_CH3/ADC123_IN2/TIM2_CH3('00'OR'01); no longer RN1A.2, RN1B.2, U2U.PA2/USART2_TX('0')/TIM5_CH3/ADC123_IN2/TIM2_CH3('00'OR'01)
- net MCU_AUX1: now also U16BANK0.IOT_215, U5U.UART4_TX/USART3_TX('01')/FT/PC10; no longer U2U.UART4_TX/USART3_TX('01')/FT/PC10, U3BANK0.IOT_215
- net MCU_AUX10: now also U16BANK2.IOB_57, U5U.PG1/FT/FSMC_A11; no longer U2U.PG1/FT/FSMC_A11, U3BANK2.IOB_57
- net MCU_AUX11: now also U16BANK2.IOB_61, U5U.FSMC_A8/FT/PF14; no longer U2U.FSMC_A8/FT/PF14, U3BANK2.IOB_61
- net MCU_AUX12: now also U16BANK2.IOB_63, U5U.FSMC_A9/FT/PF15; no longer U2U.FSMC_A9/FT/PF15, U3BANK2.IOB_63
- net MCU_AUX2: now also U16BANK0.IOT_214, U5U.UART4_RX/USART3_RX('01')/FT/PC11; no longer U2U.UART4_RX/USART3_RX('01')/FT/PC11, U3BANK0.IOT_214
- net MCU_AUX3: now also U16BANK0.IOT_213, U5U.UART5_TX/USART3_CK('01')/FT/PC12; no longer U2U.UART5_TX/USART3_CK('01')/FT/PC12, U3BANK0.IOT_213
- net MCU_AUX4: now also U16BANK0.IOT_212, U5U.PD6/FT/FSMC_NWAIT/USART2_RX('1'); no longer U2U.PD6/FT/FSMC_NWAIT/USART2_RX('1'), U3BANK0.IOT_212
- net MCU_AUX5: now also U16BANK0.IOT_206, U5U.TIM4_CH3('0')/I2C1_SCL('1')/FT/PB8; no longer U2U.TIM4_CH3('0')/I2C1_SCL('1')/FT/PB8, U3BANK0.IOT_206
- net MCU_AUX6: now also U16BANK0.IOT_192, U5U.TIM4_CH4('0')/I2C1_SDA('1')/FT/PB9; no longer U2U.TIM4_CH4('0')/I2C1_SDA('1')/FT/PB9, U3BANK0.IOT_192
- net MCU_AUX7: now also U16BANK0.IOT_191, U5U.PE0/FT/TIM4_ETR/FSMC_NBL0; no longer U2U.PE0/FT/TIM4_ETR/FSMC_NBL0, U3BANK0.IOT_191
- net MCU_AUX8: now also U16BANK0.IOT_190, U5U.PE1/FT/FSMC_NBL1; no longer U2U.PE1/FT/FSMC_NBL1, U3BANK0.IOT_190
- net MCU_AUX9: now also U16BANK2.IOB_56, U5U.FSMC_A7/FT/PF13; no longer U2U.FSMC_A7/FT/PF13, U3BANK2.IOB_56
- net MCU_INT0: now also U16BANK0.GBIN0/IOT_198, U5U.PE2/FT/FSMC_A23; no longer U2U.PE2/FT/FSMC_A23, U3BANK0.GBIN0/IOT_198
- net MCU_INT1: now also U16BANK2.GBIN5/IOB_81, U5U.PE3/FT/FSMC_A19; no longer U2U.PE3/FT/FSMC_A19, U3BANK2.GBIN5/IOB_81
- net MCU_MCO: now also U16BANK0.GBIN1/IOT_197, U5U.PA8/FT/USART1_CK/TIM1_CH1('00'OR'01')/MCO; no longer U2U.PA8/FT/USART1_CK/TIM1_CH1('00'OR'01')/MCO, U3BANK0.GBIN1/IOT_197
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Other:
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
Commit message: fix bom parts naming change back to original SC-70-5 and SC-70-6 footprints for 74LVC1G07DBV and SN74LVC1T45DBV added decoupling caps for open drain buffers(on going)
Parts:
- added C65, C66, C67, C68, C69, C70, C71, C72: 0.1uF, dp_devices.v6:CAPACITOR_NPOL-0402
- C1, C5: device rcl:C-EUC0402 -> dp_devices.v6:CAPACITOR_NPOL-0402
- C10, C11, C12, C13, C14, C15, C16, C2, C3, C4, C6, C7, C8, C9: device resistor:C-EUC0402 -> dp_devices.v6:CAPACITOR_NPOL-0402
- C17, C18, C20, C21, C22, C24, C25, C26, C27, C30, C31, C33, C34, C35, C37, C38, C40, C41, C42, C43, C44, C45, C46, C47, C48, C49, C50, C51, C52, C53, C54, C55, C56, C57, C58, C60, C61, C62, C63: device rcl:C-EUC0603 -> dp_devices.v6:CAPACITOR_NPOL-0603
- C19, C64: device rcl:CPOL-EUSMCA -> dp_devices.v6:CAPACITOR_POL-SMC_A
- C28, C39: value 1uf -> 1uF; device rcl:C-EUC0603 -> dp_devices.v6:CAPACITOR_NPOL-0603
- IC1, IC2, IC3, IC4, IC5, IC6, IC7, IC8: device dp_devices.v6:IC_BUFF_SN74LVC1T45DBV-EXTENDED -> dp_devices.v6:IC_BUFF_SN74LVC1T45DBV-SC-70-6
- R1, R10, R11, R12, R13, R14, R15, R16, R17, R18, R19, R2, R20, R21, R22, R23, R24, R3, R4, R5, R6, R7, R8, R9: device resistor:R-EU_R0402 -> dp_devices.v6:RESISTOR-0402
- R26, R29, R37, R38, R41, R42, R43, R44, R45: device rcl:R-EU_R0603 -> dp_devices.v6:RESISTOR-0603
- R33, R36, R39, R40: device resistor:R-EU_R0603 -> dp_devices.v6:RESISTOR-0603
- R46, R47, R48, R49: device dp_devices:RESISTOR-0603 -> dp_devices.v6:RESISTOR-0603
- U1, U2, U3, U4, U6, U7, U8, U9: device dp_devices.v6:IC_BUFF_74LVC1G07-EXTENDED -> dp_devices.v6:IC_BUFF_74LVC1G07
- XTAL1: device dp_devices:OSC-XTAL-12M -> dp_devices.v6:OSC-XTAL-12M
Connections:
- net 1V2: now also C31.1, C35.1, C39.2, C43.1, C54.1, C55.1; no longer C31.2, C35.2, C39.1, C43.2, C54.2, C55.2
- net 3V3: now also C1.2, C10.2, C11.2, C12.2, C17.1, C2.2, C21.1, C22.1, C25.1, C28.2, C3.2, C30.1, C33.1, C34.1, C4.2, C42.1, C44.1, C45.1, C46.1, C47.1, C48.1, C49.1, C50.1, C51.1, C52.1, C53.2, C56.1, C57.1, C58.2, C60.1, C61.2, C62.1, C63.1, C65.2, C66.2, C67.2, C68.2, C69.2, C70.2, C71.2, C72.2, C9.2; no longer C1.1, C10.1, C11.1, C12.1, C17.2, C2.1, C21.2, C22.2, C25.2, C28.1, C3.1, C30.2, C33.2, C34.2, C4.1, C42.2, C44.2, C45.2, C46.2, C47.2, C48.2, C49.2, C50.2, C51.2, C52.2, C53.1, C56.2, C57.2, C58.1, C60.2, C61.1, C62.2, C63.2, C9.1
- net GND: now also C1.1, C10.1, C11.1, C12.1, C13.2, C14.2, C15.2, C16.2, C17.2, C18.2, C2.1, C20.2, C21.2, C22.2, C24.1, C25.2, C26.1, C27.1, C28.1, C3.1, C30.2, C31.2, C33.2, C34.2, C35.2, C39.1, C4.1, C40.1, C41.1, C42.2, C43.2, C44.2, C45.2, C46.2, C47.2, C48.2, C49.2, C5.2, C50.2, C51.2, C52.2, C53.1, C54.2, C55.2, C56.2, C57.2, C58.1, C6.2, C60.2, C61.1, C62.2, C63.2, C65.1, C66.1, C67.1, C68.1, C69.1, C7.2, C70.1, C71.1, C72.1, C8.2, C9.1; no longer C1.2, C10.2, C11.2, C12.2, C13.1, C14.1, C15.1, C16.1, C17.1, C18.1, C2.2, C20.1, C21.1, C22.1, C24.2, C25.1, C26.2, C27.2, C28.2, C3.2, C30.1, C31.1, C33.1, C34.1, C35.1, C39.2, C4.2, C40.2, C41.2, C42.1, C43.1, C44.1, C45.1, C46.1, C47.1, C48.1, C49.1, C5.1, C50.1, C51.1, C52.1, C53.2, C54.1, C55.1, C56.1, C57.1, C58.2, C6.1, C60.1, C61.2, C62.1, C63.1, C7.1, C8.1, C9.2
- net N$31: now also C24.2; no longer C24.1
- net N$8: now also C20.1; no longer C20.2
- net N$9: now also C18.1; no longer C18.2
- net VREF/VOUT: now also C13.1, C14.1, C15.1, C16.1, C5.1, C6.1, C7.1, C8.1; no longer C13.2, C14.2, C15.2, C16.2, C5.2, C6.2, C7.2, C8.2
- net VUSB: now also C26.2, C27.2, C40.2, C41.2; no longer C26.1, C27.1, C40.1, C41.1
Other:
- moved on the sheet: C59, U1P, U2P, U4P, U6P, U7P, U8P, U9P

Commit message: Revert previous commit to v1b, wrong version commited. changes should be on v1c not v1b.
This reverts commit d10a26b079303959180bb4ab2616075854f9b9d1.
Parts:
- removed C65, C66, C67, C68, C69, C70, C71, C72: 0.1uF, dp_devices.v6:CAPACITOR_NPOL-0402
- C1, C5: device dp_devices.v6:CAPACITOR_NPOL-0402 -> rcl:C-EUC0402
- C10, C11, C12, C13, C14, C15, C16, C2, C3, C4, C6, C7, C8, C9: device dp_devices.v6:CAPACITOR_NPOL-0402 -> resistor:C-EUC0402
- C17, C18, C20, C21, C22, C24, C25, C26, C27, C30, C31, C33, C34, C35, C37, C38, C40, C41, C42, C43, C44, C45, C46, C47, C48, C49, C50, C51, C52, C53, C54, C55, C56, C57, C58, C60, C61, C62, C63: device dp_devices.v6:CAPACITOR_NPOL-0603 -> rcl:C-EUC0603
- C19, C64: device dp_devices.v6:CAPACITOR_POL-SMC_A -> rcl:CPOL-EUSMCA
- C28, C39: value 1uF -> 1uf; device dp_devices.v6:CAPACITOR_NPOL-0603 -> rcl:C-EUC0603
- IC1, IC2, IC3, IC4, IC5, IC6, IC7, IC8: device dp_devices.v6:IC_BUFF_SN74LVC1T45DBV-SC-70-6 -> dp_devices.v6:IC_BUFF_SN74LVC1T45DBV-EXTENDED
- R1, R10, R11, R12, R13, R14, R15, R16, R17, R18, R19, R2, R20, R21, R22, R23, R24, R3, R4, R5, R6, R7, R8, R9: device dp_devices.v6:RESISTOR-0402 -> resistor:R-EU_R0402
- R26, R29, R37, R38, R41, R42, R43, R44, R45: device dp_devices.v6:RESISTOR-0603 -> rcl:R-EU_R0603
- R33, R36, R39, R40: device dp_devices.v6:RESISTOR-0603 -> resistor:R-EU_R0603
- R46, R47, R48, R49: device dp_devices.v6:RESISTOR-0603 -> dp_devices:RESISTOR-0603
- U1, U2, U3, U4, U6, U7, U8, U9: device dp_devices.v6:IC_BUFF_74LVC1G07 -> dp_devices.v6:IC_BUFF_74LVC1G07-EXTENDED
- XTAL1: device dp_devices.v6:OSC-XTAL-12M -> dp_devices:OSC-XTAL-12M
Connections:
- net 1V2: now also C31.2, C35.2, C39.1, C43.2, C54.2, C55.2; no longer C31.1, C35.1, C39.2, C43.1, C54.1, C55.1
- net 3V3: now also C1.1, C10.1, C11.1, C12.1, C17.2, C2.1, C21.2, C22.2, C25.2, C28.1, C3.1, C30.2, C33.2, C34.2, C4.1, C42.2, C44.2, C45.2, C46.2, C47.2, C48.2, C49.2, C50.2, C51.2, C52.2, C53.1, C56.2, C57.2, C58.1, C60.2, C61.1, C62.2, C63.2, C9.1; no longer C1.2, C10.2, C11.2, C12.2, C17.1, C2.2, C21.1, C22.1, C25.1, C28.2, C3.2, C30.1, C33.1, C34.1, C4.2, C42.1, C44.1, C45.1, C46.1, C47.1, C48.1, C49.1, C50.1, C51.1, C52.1, C53.2, C56.1, C57.1, C58.2, C60.1, C61.2, C62.1, C63.1, C65.2, C66.2, C67.2, C68.2, C69.2, C70.2, C71.2, C72.2, C9.2
- net GND: now also C1.2, C10.2, C11.2, C12.2, C13.1, C14.1, C15.1, C16.1, C17.1, C18.1, C2.2, C20.1, C21.1, C22.1, C24.2, C25.1, C26.2, C27.2, C28.2, C3.2, C30.1, C31.1, C33.1, C34.1, C35.1, C39.2, C4.2, C40.2, C41.2, C42.1, C43.1, C44.1, C45.1, C46.1, C47.1, C48.1, C49.1, C5.1, C50.1, C51.1, C52.1, C53.2, C54.1, C55.1, C56.1, C57.1, C58.2, C6.1, C60.1, C61.2, C62.1, C63.1, C7.1, C8.1, C9.2; no longer C1.1, C10.1, C11.1, C12.1, C13.2, C14.2, C15.2, C16.2, C17.2, C18.2, C2.1, C20.2, C21.2, C22.2, C24.1, C25.2, C26.1, C27.1, C28.1, C3.1, C30.2, C31.2, C33.2, C34.2, C35.2, C39.1, C4.1, C40.1, C41.1, C42.2, C43.2, C44.2, C45.2, C46.2, C47.2, C48.2, C49.2, C5.2, C50.2, C51.2, C52.2, C53.1, C54.2, C55.2, C56.2, C57.2, C58.1, C6.2, C60.2, C61.1, C62.2, C63.2, C65.1, C66.1, C67.1, C68.1, C69.1, C7.2, C70.1, C71.1, C72.1, C8.2, C9.1
- net N$31: now also C24.1; no longer C24.2
- net N$8: now also C20.2; no longer C20.1
- net N$9: now also C18.2; no longer C18.1
- net VREF/VOUT: now also C13.2, C14.2, C15.2, C16.2, C5.2, C6.2, C7.2, C8.2; no longer C13.1, C14.1, C15.1, C16.1, C5.1, C6.1, C7.1, C8.1
- net VUSB: now also C26.1, C27.1, C40.1, C41.1; no longer C26.2, C27.2, C40.2, C41.2
Other:
- moved on the sheet: C59, U1P, U2P, U4P, U6P, U7P, U8P, U9P
