File: BPUv1c/BusPirate-ultra.v1.0c.brd (EAGLE design)
At the start: 100 x 50 mm, 187 parts, among them J1 USB-C-12, J2 CON_HEADER_1X04, J3 CON_HEADER_1X10-RIGHT_ANGLED_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, J4 CON_MOLEX_MALE_SMT_SH_1.25, Q300 PMV65XP, Q301 DMMT3906W, U100 STM32F103ZX, U101 W25X40CL, U200 74HCT4067, U201 MCP6001, U202 ADS7041, U300 MCP1824_ADJ, U301 MCP6001, U302 MCP1700, U303 MCP1801T-1202I/OT, U400 SN74LVC1T45DBV, U401 SN74LVC1T45DBV, U402 74LVC1G07DBV, U403 74LVC1G07DBV, U404 SN74LVC1T45DBV, U405 SN74LVC1T45DBV, U406 74LVC1G07DBV, U407 74LVC1G07DBV, U408 SN74LVC1T45DBV, U409 SN74LVC1T45DBV, U410 74LVC1G07DBV, U411 74LVC1G07DBV, U412 SN74LVC1T45DBV, U413 SN74LVC1T45DBV, U414 74LVC1G07DBV, U415 74LVC1G07DBV, U500 74HCT4066PW, U501 74HCT4066PW, U600 23LC1024, U601 23LC1024, U602 74LVC245A, U700 ICE40HX4K

Commit message: change supply of ADC chip to 3.3V
Connections:
- net 3V3: now also C204.1, C205.1, U202.1, U202.7
- net VUSB: no longer C204.1, C205.1, U202.1, U202.7
Changed lines of the file:
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@@
 <wire x1="26.8106" y1="41.8728" x2="27.94" y2="43.0022" width="0.4064" layer="1"/>
 <contactref element="U302" pad="3"/>
+<contactref element="U202" pad="7"/>
+<contactref element="C204" pad="1"/>
+<contactref element="U202" pad="1"/>
+<contactref element="C205" pad="1"/>
 <wire x1="36.785" y1="35.351" x2="39.79" y2="36.3728" width="0" layer="19" extent="1-1"/>
-<wire x1="-24.408" y1="-46.608" x2="19.501" y2="4.477" width="0" layer="19" extent="1-1"/>
+<wire x1="-16.506" y1="-32.486" x2="19.501" y2="4.477" width="0" layer="19" extent="1-1"/>
+<wire x1="-17.006" y1="-35.586" x2="-16.506" y2="-32.486" width="0" layer="19" extent="1-1"/>
+<wire x1="-17.106" y1="-41.402" x2="-17.006" y2="-35.586" width="0" layer="19" extent="1-1"/>
+<wire x1="-17.106" y1="-47.498" x2="-17.106" y2="-41.402" width="0" layer="19" extent="1-1"/>
+<wire x1="-24.408" y1="-46.608" x2="-17.106" y2="-47.498" width="0" layer="19" extent="1-1"/>
 </signal>
 <signal name="N$7">
@@
 <contactref element="C305" pad="2"/>
 <contactref element="C307" pad="2"/>
-<contactref element="U202" pad="7"/>
-<contactref element="C204" pad="1"/>
-<contactref element="U202" pad="1"/>
-<contactref element="C205" pad="1"/>
 <contactref element="U302" pad="2"/>
 <contactref element="C200" pad="2"/>
@@
 <wire x1="-7.532" y1="-17.018" x2="9.7638" y2="4.6436" width="0" layer="19" extent="1-1"/>
 <wire x1="-7.532" y1="-23.114" x2="-7.532" y2="-17.018" width="0" layer="19" extent="1-1"/>
-<wire x1="-16.506" y1="-32.486" x2="-7.532" y2="-23.114" width="0" layer="19" extent="1-1"/>
-<wire x1="-17.006" y1="-35.586" x2="-16.506" y2="-32.486" width="0" layer="19" extent="1-1"/>
-<wire x1="-17.106" y1="-41.402" x2="-17.006" y2="-35.586" width="0" layer="19" extent="1-1"/>
-<wire x1="-17.106" y1="-47.498" x2="-17.106" y2="-41.402" width="0" layer="19" extent="1-1"/>
-<wire x1="-25.908" y1="-45.108" x2="-17.106" y2="-47.498" width="0" layer="19" extent="1-1"/>
+<wire x1="-25.908" y1="-45.108" x2="-7.532" y2="-23.114" width="0" layer="19" extent="1-1"/>
 <wire x1="-28.99" y1="-52.7082" x2="-25.908" y2="-45.108" width="0" layer="19" extent="1-1"/>
 </signal>

Commit message: updates on v1c schematic moved MCU_VPU to PA9, free up A10 moved DISPLAY_CS to PF11 (former DISPLAY_D/P) and DISPLAY_D/P to PB1, free up A6 moved FPGA MCU_INT1 from GBIN5 to FPGA pin 115 wired PG8 to FPGA GBIN6 (former FPGA PWM) as MASTER_RESET wired PWM pin (MCU pin PC6) to FPGA GBIN5, this new trace is long compared to old moved MCU_INT0 from MCU PE2 to PA10 moved MCU_INT1 from MCU PE3 to PC9 MCU PE2 to PE4 are now freed
Connections:
- removed net N$41: U100.99
- removed net N$53: U100.93
- removed net UART_RX: U100.102
- removed net UART_TX: U100.101
- new net MASTER_RESET: U100.93, U700.21
- new net N$48: U100.136
- new net N$49: U100.137
- new net N$50: U700.20
- new net N$51: U700.52
- net DISPLAY_CS: now also U100.49; no longer U100.50
- net DISPLAY_D/P: now also U100.47; no longer U100.49
- net MCU_INT0: now also U100.102; no longer U100.1
- net MCU_INT1: now also U100.99, U700.115; no longer U100.2, U700.49
- net MCU_VPU: now also U100.101; no longer U100.56
- net PWM: now also U700.49; no longer U700.21
Routing:
- net MCU_INT1: track 64.3 -> 0.00 mm, vias 2 -> 0
- net MCU_INT0: track 42.7 -> 33.8 mm
- net DISPLAY_D/P: track 11.8 -> 7.78 mm
- net DISPLAY_CS: track 12.1 -> 8.28 mm
- net PWM: track 9.62 -> 6.98 mm
- net MCU_VPU: track 119.3 -> 118.7 mm
Changed lines of the file:
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@@
 <wire x1="34.785" y1="35.75" x2="34.785" y2="36.131" width="0.254" layer="1"/>
-</signal>
-<signal name="UART_RX">
-<contactref element="U100" pad="102"/>
-</signal>
-<signal name="UART_TX">
-<contactref element="U100" pad="101"/>
 </signal>
 <signal name="D+">
@@
 <via x="52.832" y="36.9288" extent="1-16" drill="0.508"/>
 <wire x1="28.6738" y1="39.3418" x2="48.387" y2="39.3418" width="0.254" layer="16"/>
-<contactref element="U100" pad="1"/>
-<wire x1="15.285" y1="33.75" x2="24.225" y2="33.75" width="0.254" layer="1"/>
 <wire x1="24.765" y1="34.29" x2="24.225" y2="33.75" width="0.254" layer="1"/>
 <wire x1="28.6738" y1="39.3418" x2="24.765" y2="35.433" width="0.254" layer="16"/>
@@
 <wire x1="52.8393" y1="36.766" x2="52.8393" y2="35.75" width="0.254" layer="1"/>
 <wire x1="52.832" y1="36.9288" x2="52.832" y2="36.7733" width="0.254" layer="1"/>
+<contactref element="U100" pad="102"/>
+<wire x1="28.6738" y1="39.3418" x2="36.785" y2="30.75" width="0" layer="19" extent="1-16"/>
 </signal>
 <signal name="MCU_INT1">
-<via x="25.654" y="33.909" extent="1-16" drill="0.4064"/>
-<wire x1="28.8167375" y1="38.91" x2="48.133" y2="38.91" width="0.254" layer="16"/>
-<contactref element="U100" pad="2"/>
-<wire x1="15.285" y1="33.25" x2="24.995" y2="33.25" width="0.254" layer="1"/>
-<wire x1="28.8167375" y1="38.91" x2="25.654" y2="35.7472625" width="0.254" layer="16"/>
-<wire x1="24.995" y1="33.25" x2="25.654" y2="33.909" width="0.254" layer="1"/>
-<wire x1="25.654" y1="35.7472625" x2="25.654" y2="33.909" width="0.254" layer="16"/>
-<wire x1="53.848" y1="30.353" x2="51.435" y2="27.94" width="0.254" layer="16"/>
-<wire x1="48.133" y1="38.91" x2="53.848" y2="33.195" width="0.254" layer="16"/>
-<wire x1="53.848" y1="33.195" x2="53.848" y2="30.353" width="0.254" layer="16"/>
-<contactref element="U700" pad="49"/>
-<wire x1="51.3393" y1="14.25" x2="51.3393" y2="16.5413" width="0.254" layer="1"/>
-<wire x1="51.3393" y1="16.5413" x2="51.435" y2="16.637" width="0.254" layer="1"/>
-<via x="51.435" y="16.637" extent="1-16" drill="0.4064"/>
-<wire x1="51.435" y1="16.637" x2="51.435" y2="27.94" width="0.254" layer="16"/>
+<contactref element="U700" pad="115"/>
+<contactref element="U100" pad="99"/>
+<wire x1="36.785" y1="29.25" x2="59.8393" y2="35.75" width="0" layer="19" extent="1-1"/>
 </signal>
 <signal name="PWM">
-<contactref element="U700" pad="21"/>
 <contactref element="U100" pad="96"/>
 <wire x1="40.6964625" y1="23.75" x2="39.7684" y2="24.6780625" width="0.254" layer="1"/>
@@
 <wire x1="39.7684" y1="27.09073125" x2="39.10913125" y2="27.75" width="0.254" layer="1"/>
 <wire x1="39.10913125" y1="27.75" x2="36.785" y2="27.75" width="0.254" layer="1"/>
-<wire x1="43.3393" y1="23.75" x2="40.6964625" y2="23.75" width="0.254" layer="1"/>
+<contactref element="U700" pad="49"/>
+<wire x1="40.6964625" y1="23.75" x2="51.3393" y2="14.25" width="0" layer="19" extent="1-1"/>
 </signal>
 <signal name="MCU_MCO">
@@
 <contactref element="U100" pad="27"/>
 </signal>
-<signal name="N$41">
-<contactref element="U100" pad="99"/>
-</signal>
 <signal name="N$23">
 <contactref element="U100" pad="28"/>
@@
 <contactref element="U100" pad="90"/>
 </signal>
-<signal name="N$53">
+<signal name="MASTER_RESET">
 <contactref element="U100" pad="93"/>
+<contactref element="U700" pad="21"/>
+<wire x1="36.785" y1="26.25" x2="43.3393" y2="23.75" width="0" layer="19" extent="1-1"/>
 </signal>
 <signal name="N$54">
@@
 <contactref element="U501" pad="5"/>
 <contactref element="U501" pad="6"/>
-<contactref element="U100" pad="56"/>
 <wire x1="90.2" y1="3.65" x2="89.55" y2="3.65" width="0.254" layer="1"/>
 <wire x1="88.25" y1="9.25" x2="87.6" y2="9.25" width="0.254" layer="1"/>
@@
 <via x="87.63" y="7.874" extent="1-16" drill="0.35"/>
 <wire x1="87.63" y1="7.874" x2="91.059" y2="11.303" width="0.3048" layer="16"/>
-<wire x1="26.785" y1="14.25" x2="26.785" y2="13.601" width="0.254" layer="1"/>
 <wire x1="26.785" y1="13.601" x2="27.432" y2="12.954" width="0.254" layer="1"/>
 <via x="27.432" y="12.954" extent="1-16" drill="0.4064"/>
@@
 <wire x1="61.214" y1="7.112" x2="63.3984" y2="4.9276" width="0.254" layer="1"/>
 <wire x1="63.3984" y1="4.9276" x2="63.5" y2="4.9276" width="0.254" layer="1"/>
+<contactref element="U100" pad="101"/>
+<wire x1="36.8172375" y1="12.2936" x2="36.785" y2="30.25" width="0" layer="19" extent="1-16"/>
 </signal>
 <signal name="DISPLAY_SPI_CLOCK">
@@
 <signal name="DISPLAY_CS">
 <contactref element="J4" pad="P1"/>
-<contactref element="U100" pad="50"/>
 <wire x1="23.785" y1="10.38813125" x2="29.501" y2="4.67213125" width="0.254" layer="1"/>
-<wire x1="23.785" y1="14.25" x2="23.785" y2="10.38813125" width="0.254" layer="1"/>
 <wire x1="29.501" y1="4.67213125" x2="29.501" y2="4.477" width="0.254" layer="1"/>
+<contactref element="U100" pad="49"/>
+<wire x1="23.785" y1="10.38813125" x2="23.285" y2="14.25" width="0" layer="19" extent="1-1"/>
 </signal>
 <signal name="DISPLAY_D/P">
 <contactref element="J4" pad="P2"/>
-<contactref element="U100" pad="49"/>
-<wire x1="23.285" y1="14.25" x2="23.285" y2="10.205" width="0.254" layer="1"/>
 <wire x1="23.285" y1="10.205" x2="28.251" y2="5.239" width="0.254" layer="1"/>
 <wire x1="28.251" y1="5.239" x2="28.251" y2="4.477" width="0.254" layer="1"/>
+<contactref element="U100" pad="47"/>
+<wire x1="23.285" y1="10.205" x2="22.285" y2="14.25" width="0" layer="19" extent="1-1"/>
 </signal>
 <signal name="DISPLAY_PWM">
@@
 <wire x1="58.039" y1="5.295" x2="-28.99" y2="-58.5438" width="0" layer="19" extent="1-1"/>
 </signal>
+<signal name="N$48">
+<contactref element="U100" pad="136"/>
+</signal>
+<signal name="N$49">
+<contactref element="U100" pad="137"/>
+</signal>
+<signal name="N$50">
+<contactref element="U700" pad="20"/>
+</signal>
+<signal name="N$51">
+<contactref element="U700" pad="52"/>
+</signal>
 </signals>
