File: BPUv1c/BusPirate-ultra.v1.0c.sch (EAGLE design)
At the start: 184 parts, among them J1 USB-C-12, J2 CON_HEADER_1X04, J3 CON_HEADER_1X10-RIGHT_ANGLED_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, J4 CON_MOLEX_MALE_SMT_SH_1.25, Q300 PMV65XP, Q301 DMMT3906W, U100 STM32F103ZX, U101 W25X40CL, U200 74HCT4067, U201 MCP6001, U202 ADS7041, U300 MCP1824_ADJ, U301 MCP6001, U302 MCP1700, U303 MCP1801T-1202I/OT, U400 SN74LVC1T45DBV, U401 SN74LVC1T45DBV, U402 74LVC1G07DBV, U403 74LVC1G07DBV, U404 SN74LVC1T45DBV, U405 SN74LVC1T45DBV, U406 74LVC1G07DBV, U407 74LVC1G07DBV, U408 SN74LVC1T45DBV, U409 SN74LVC1T45DBV, U410 74LVC1G07DBV, U411 74LVC1G07DBV, U412 SN74LVC1T45DBV, U413 SN74LVC1T45DBV, U414 74LVC1G07DBV, U415 74LVC1G07DBV, U500 74HCT4066PW, U501 74HCT4066PW, U600 23LC1024, U601 23LC1024, U602 74LVC245A, U700 ICE40HX4K

Commit message: updates on v1c schematic moved MCU_VPU to PA9, free up A10 moved DISPLAY_CS to PF11 (former DISPLAY_D/P) and DISPLAY_D/P to PB1, free up A6 moved FPGA MCU_INT1 from GBIN5 to FPGA pin 115 wired PG8 to FPGA GBIN6 (former FPGA PWM) as MASTER_RESET wired PWM pin (MCU pin PC6) to FPGA GBIN5, this new trace is long compared to old moved MCU_INT0 from MCU PE2 to PA10 moved MCU_INT1 from MCU PE3 to PC9 MCU PE2 to PE4 are now freed
Connections:
- removed net N$41: U100U.TIM8_CH4/TIM3_CH4('11')/FT/PC9
- removed net N$53: U100U.PG8/FT
- removed net UART_RX: U100U.PA10/FT/USART1_RX('0')/TIM1_CH3('00'OR'01')
- removed net UART_TX: U100U.PA9/FT/USART1_TX('0')/TIM1_CH2('00'OR'01')
- new net MASTER_RESET: U100U.PG8/FT, U700BANK3.GBIN6/IOL_14A
- new net N$48: U100U.I2C1_SCL('0')/TIM4_CH1('0')/USART1_TX('1')/FT/PB6
- new net N$49: U100U.I2C1_SDA('0')/FSMC_NADV/TIM4_CH2('0')/USART1_RX('1')/FT/PB7
- new net N$50: U700BANK3.GBIN7/IOL_13B
- new net N$51: U700BANK2.GBIN4/IOB_82
- net DISPLAY_CS: now also U100U.FSMC_NIOS16/FT/PF11; no longer U100U.FSMC_A6/FT/PF12
- net DISPLAY_D/P: now also U100U.ADC12_IN9/TIM3_CH4('00'OR'10')/TIM8_CH3N/TIM1_CH3N('01')/PB1; no longer U100U.FSMC_NIOS16/FT/PF11
- net MCU_INT0: now also U100U.PA10/FT/USART1_RX('0')/TIM1_CH3('00'OR'01'); no longer U100U.PE2/FT/FSMC_A23
- net MCU_INT1: now also U100U.TIM8_CH4/TIM3_CH4('11')/FT/PC9, U700BANK0.IOT_172; no longer U100U.PE3/FT/FSMC_A19, U700BANK2.GBIN5/IOB_81
- net MCU_VPU: now also U100U.PA9/FT/USART1_TX('0')/TIM1_CH2('00'OR'01'); no longer U100U.PG0/FT/FSMC_A10
- net PWM: now also U700BANK2.GBIN5/IOB_81; no longer U700BANK3.GBIN6/IOL_14A
Changed lines of the file:
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@@
-</segment>
-</net>
-<net name="UART_RX" class="0">
-<segment>
-<pinref part="U100" gate="U" pin="PA10/FT/USART1_RX('0')/TIM1_CH3('00'OR'01')"/>
-<wire x1="73.66" y1="447.04" x2="71.12" y2="447.04" width="0.1524" layer="91"/>
-<label x="71.12" y="447.04" size="1.778" layer="95" align="center-right"/>
-</segment>
-</net>
-<net name="UART_TX" class="0">
-<segment>
-<pinref part="U100" gate="U" pin="PA9/FT/USART1_TX('0')/TIM1_CH2('00'OR'01')"/>
-<wire x1="73.66" y1="449.58" x2="71.12" y2="449.58" width="0.1524" layer="91"/>
-<label x="71.12" y="449.58" size="1.778" layer="95" align="center-right"/>
 </segment>
 </net>
@@
 </segment>
 <segment>
-<pinref part="U100" gate="U" pin="PE2/FT/FSMC_A23"/>
-<wire x1="73.66" y1="381" x2="71.12" y2="381" width="0.1524" layer="91"/>
-<label x="71.12" y="381" size="1.778" layer="95" align="center-right"/>
+<pinref part="U100" gate="U" pin="PA10/FT/USART1_RX('0')/TIM1_CH3('00'OR'01')"/>
+<wire x1="73.66" y1="447.04" x2="71.12" y2="447.04" width="0.1524" layer="91"/>
+<label x="71.12" y="447.04" size="1.778" layer="95" align="center-right"/>
 </segment>
 </net>
 <net name="MCU_INT1" class="0">
 <segment>
-<pinref part="U100" gate="U" pin="PE3/FT/FSMC_A19"/>
-<wire x1="73.66" y1="378.46" x2="71.12" y2="378.46" width="0.1524" layer="91"/>
-<label x="71.12" y="378.46" size="1.778" layer="95" align="center-right"/>
-</segment>
-<segment>
-<pinref part="U700" gate="BANK2" pin="GBIN5/IOB_81"/>
-<wire x1="528.32" y1="45.72" x2="530.86" y2="45.72" width="0.1524" layer="91"/>
-<label x="530.86" y="45.72" size="1.778" layer="95" align="center-left"/>
+<pinref part="U700" gate="BANK0" pin="IOT_172"/>
+<wire x1="391.16" y1="142.24" x2="388.62" y2="142.24" width="0.1524" layer="91"/>
+<label x="388.62" y="142.24" size="1.778" layer="95" align="center-right"/>
+</segment>
+<segment>
+<pinref part="U100" gate="U" pin="TIM8_CH4/TIM3_CH4('11')/FT/PC9"/>
+<wire x1="180.34" y1="406.4" x2="182.88" y2="406.4" width="0.1524" layer="91"/>
+<label x="182.88" y="406.4" size="1.778" layer="95"/>
 </segment>
 </net>
 <net name="PWM" class="0">
-<segment>
-<pinref part="U700" gate="BANK3" pin="GBIN6/IOL_14A"/>
-<wire x1="429.26" y1="60.96" x2="431.8" y2="60.96" width="0.1524" layer="91"/>
-<label x="431.8" y="60.96" size="1.778" layer="95" align="center-left"/>
-</segment>
 <segment>
 <pinref part="U100" gate="U" pin="TIM8_CH1/TIM3_CH1('11')/FT/PC6"/>
 <wire x1="180.34" y1="414.02" x2="182.88" y2="414.02" width="0.1524" layer="91"/>
 <label x="182.88" y="414.02" size="1.778" layer="95" align="center-left"/>
+</segment>
+<segment>
+<pinref part="U700" gate="BANK2" pin="GBIN5/IOB_81"/>
+<wire x1="528.32" y1="45.72" x2="530.86" y2="45.72" width="0.1524" layer="91"/>
+<label x="530.86" y="45.72" size="1.778" layer="95"/>
 </segment>
 </net>
@@
 </segment>
 </net>
-<net name="N$41" class="0">
-<segment>
-<pinref part="U100" gate="U" pin="TIM8_CH4/TIM3_CH4('11')/FT/PC9"/>
-<wire x1="180.34" y1="406.4" x2="182.88" y2="406.4" width="0.1524" layer="91"/>
-</segment>
-</net>
 <net name="N$23" class="0">
 <segment>
@@
 <segment>
 <pinref part="U700" gate="BANK0" pin="IOT_181"/>
-<wire x1="426.72" y1="139.7" x2="429.26" y2="139.7" width="0.1524" layer="91"/>
-<label x="429.26" y="139.7" size="1.778" layer="95" align="center-left"/>
+<wire x1="426.72" y1="139.7" x2="431.8" y2="139.7" width="0.1524" layer="91"/>
+<label x="431.8" y="139.7" size="1.778" layer="95" align="center-left"/>
 </segment>
 </net>
@@
 <segment>
 <pinref part="U700" gate="BANK0" pin="IOT_178"/>
-<wire x1="426.72" y1="134.62" x2="429.26" y2="134.62" width="0.1524" layer="91"/>
-<label x="429.26" y="134.62" size="1.778" layer="95" align="center-left"/>
+<wire x1="426.72" y1="134.62" x2="431.8" y2="134.62" width="0.1524" layer="91"/>
+<label x="431.8" y="134.62" size="1.778" layer="95" align="center-left"/>
 </segment>
 </net>
@@
 <segment>
 <pinref part="U700" gate="BANK0" pin="IOT_179"/>
-<wire x1="426.72" y1="137.16" x2="429.26" y2="137.16" width="0.1524" layer="91"/>
-<label x="429.26" y="137.16" size="1.778" layer="95" align="center-left"/>
+<wire x1="426.72" y1="137.16" x2="431.8" y2="137.16" width="0.1524" layer="91"/>
+<label x="431.8" y="137.16" size="1.778" layer="95" align="center-left"/>
 </segment>
 </net>
@@
 </segment>
 </net>
-<net name="N$53" class="0">
+<net name="MASTER_RESET" class="0">
 <segment>
 <pinref part="U100" gate="U" pin="PG8/FT"/>
 <wire x1="73.66" y1="322.58" x2="71.12" y2="322.58" width="0.1524" layer="91"/>
+<label x="71.12" y="322.58" size="1.778" layer="95" align="center-right"/>
+</segment>
+<segment>
+<pinref part="U700" gate="BANK3" pin="GBIN6/IOL_14A"/>
+<wire x1="429.26" y1="60.96" x2="431.8" y2="60.96" width="0.1524" layer="91"/>
+<label x="431.8" y="60.96" size="1.778" layer="95" align="center-left"/>
 </segment>
 </net>
@@
 <segment>
 <pinref part="U700" gate="BANK1" pin="GBIN3/IOR_140"/>
-<wire x1="528.32" y1="147.32" x2="530.86" y2="147.32" width="0.1524" layer="91"/>
-<label x="530.86" y="147.32" size="1.778" layer="95"/>
+<wire x1="528.32" y1="147.32" x2="533.4" y2="147.32" width="0.1524" layer="91"/>
+<label x="533.4" y="147.32" size="1.778" layer="95"/>
 </segment>
 <segment>
@@
 <segment>
 <pinref part="U700" gate="BANK1" pin="GBIN2/IOR_141"/>
-<wire x1="528.32" y1="149.86" x2="530.86" y2="149.86" width="0.1524" layer="91"/>
-<label x="530.86" y="149.86" size="1.778" layer="95"/>
+<wire x1="528.32" y1="149.86" x2="533.4" y2="149.86" width="0.1524" layer="91"/>
+<label x="533.4" y="149.86" size="1.778" layer="95"/>
 </segment>
 <segment>
@@
 <segment>
 <pinref part="U700" gate="BANK1" pin="IOR_144"/>
-<wire x1="528.32" y1="152.4" x2="530.86" y2="152.4" width="0.1524" layer="91"/>
-<label x="530.86" y="152.4" size="1.778" layer="95"/>
+<wire x1="528.32" y1="152.4" x2="533.4" y2="152.4" width="0.1524" layer="91"/>
+<label x="533.4" y="152.4" size="1.778" layer="95"/>
 </segment>
 <segment>
@@
 <segment>
 <pinref part="U700" gate="BANK1" pin="IOR_146"/>
-<wire x1="528.32" y1="154.94" x2="530.86" y2="154.94" width="0.1524" layer="91"/>
-<label x="530.86" y="154.94" size="1.778" layer="95"/>
+<wire x1="528.32" y1="154.94" x2="533.4" y2="154.94" width="0.1524" layer="91"/>
+<label x="533.4" y="154.94" size="1.778" layer="95"/>
 </segment>
 <segment>
@@
 </segment>
 <segment>
-<pinref part="U100" gate="U" pin="PG0/FT/FSMC_A10"/>
-<wire x1="73.66" y1="342.9" x2="71.12" y2="342.9" width="0.1524" layer="91"/>
-<label x="71.12" y="342.9" size="1.778" layer="95" align="center-right"/>
+<pinref part="U100" gate="U" pin="PA9/FT/USART1_TX('0')/TIM1_CH2('00'OR'01')"/>
+<wire x1="73.66" y1="449.58" x2="71.12" y2="449.58" width="0.1524" layer="91"/>
+<label x="71.12" y="449.58" size="1.778" layer="95" align="center-right"/>
 </segment>
 </net>
@@
 </segment>
 <segment>
-<pinref part="U100" gate="U" pin="FSMC_A6/FT/PF12"/>
-<wire x1="180.34" y1="355.6" x2="182.88" y2="355.6" width="0.1524" layer="91"/>
-<label x="182.88" y="355.6" size="1.778" layer="95" align="center-left"/>
+<pinref part="U100" gate="U" pin="FSMC_NIOS16/FT/PF11"/>
+<wire x1="180.34" y1="358.14" x2="182.88" y2="358.14" width="0.1524" layer="91"/>
+<label x="182.88" y="358.14" size="1.778" layer="95" align="center-left"/>
 </segment>
 </net>
@@
 </segment>
 <segment>
-<pinref part="U100" gate="U" pin="FSMC_NIOS16/FT/PF11"/>
-<wire x1="180.34" y1="358.14" x2="182.88" y2="358.14" width="0.1524" layer="91"/>
-<label x="182.88" y="358.14" size="1.778" layer="95" align="center-left"/>
+<pinref part="U100" gate="U" pin="ADC12_IN9/TIM3_CH4('00'OR'10')/TIM8_CH3N/TIM1_CH3N('01')/PB1"/>
+<wire x1="180.34" y1="340.36" x2="182.88" y2="340.36" width="0.1524" layer="91"/>
+<label x="182.88" y="340.36" size="1.778" layer="95"/>
 </segment>
 </net>
@@
 </segment>
 </net>
+<net name="N$48" class="0">
+<segment>
+<pinref part="U100" gate="U" pin="I2C1_SCL('0')/TIM4_CH1('0')/USART1_TX('1')/FT/PB6"/>
+<wire x1="180.34" y1="327.66" x2="182.88" y2="327.66" width="0.1524" layer="91"/>
+</segment>
+</net>
+<net name="N$49" class="0">
+<segment>
+<pinref part="U100" gate="U" pin="I2C1_SDA('0')/FSMC_NADV/TIM4_CH2('0')/USART1_RX('1')/FT/PB7"/>
+<wire x1="180.34" y1="325.12" x2="182.88" y2="325.12" width="0.1524" layer="91"/>
+</segment>
+</net>
+<net name="N$50" class="0">
+<segment>
+<pinref part="U700" gate="BANK3" pin="GBIN7/IOL_13B"/>
+<wire x1="429.26" y1="58.42" x2="431.8" y2="58.42" width="0.1524" layer="91"/>
+</segment>
+</net>
+<net name="N$51" class="0">
+<segment>
+<pinref part="U700" gate="BANK2" pin="GBIN4/IOB_82"/>
+<wire x1="528.32" y1="48.26" x2="530.86" y2="48.26" width="0.1524" layer="91"/>
+</segment>
+</net>

Commit message: renamed DISPLAY_AUX2 to DISPLAY_AUX1 connected to PB1 renamed DISPLAY_AUX1 to DISPLAY_RESET and connected to PB2/BOOT1, wired a pull down resistor too rewired DISPLAY_CS from PF11 to PC4 rewired DISPLAY_D/P from PB1 to PC5 wired FSMC_A6/PF12 to FPGA pin 42 renamed MCU_AUX9 to FSMC_A7 renamed MCU_AUX11 to FSMC_A8 renamed MCU_AUX12 to FSMC_A9 renamed MCU_AUX10 to FSMC_A10 and move it to FSMC_A10/PG0 wired PG1/MCU_INT2 to FPGA pin 114
Parts:
- added R101: 10K, dp_devices.v6:RESISTOR-0402
Connections:
- net MCU_AUX11 renamed FSMC_A8
- net MCU_AUX12 renamed FSMC_A9
- net MCU_AUX9 renamed FSMC_A7
- removed net DISPLAY_AUX2: J4.4, U100U.ADC12_IN15/PC5
- removed net MCU_AUX10: U100U.PG1/FT/FSMC_A11, U700BANK2.IOB_57
- new net DISPLAY_RESET: J4.5, R101.2, U100U.BOOT1/FT/PB2
- new net FSMC_A10: U100U.PG0/FT/FSMC_A10, U700BANK2.IOB_57
- new net FSMC_A6: U100U.FSMC_A6/FT/PF12, U700BANK2.IOB_64
- new net MCU_INT2: U100U.PG1/FT/FSMC_A11, U700BANK0.IOT_171
- new net N$10: U100U.FSMC_NIOS16/FT/PF11
- net DISPLAY_AUX1: now also J4.4, U100U.ADC12_IN9/TIM3_CH4('00'OR'10')/TIM8_CH3N/TIM1_CH3N('01')/PB1; no longer J4.5, U100U.ADC12_IN14/PC4
- net DISPLAY_CS: now also U100U.ADC12_IN14/PC4; no longer U100U.FSMC_NIOS16/FT/PF11
- net DISPLAY_D/P: now also U100U.ADC12_IN15/PC5; no longer U100U.ADC12_IN9/TIM3_CH4('00'OR'10')/TIM8_CH3N/TIM1_CH3N('01')/PB1
- net GND: now also R101.1; no longer U100U.BOOT1/FT/PB2
Changed lines of the file:
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@@
 <part name="U200" library="dp_devices.v6" deviceset="IC_74HCT4067" device="" value="74HCT4067"/>
 <part name="SUPPLY41" library="supply2" deviceset="V+" device=""/>
+<part name="R101" library="dp_devices.v6" deviceset="RESISTOR" device="-0402" value="10K"/>
 </parts>
 <sheets>
@@
 <instance part="GND61" gate="G$1" x="472.44" y="411.48" smashed="yes"/>
 <instance part="GND33" gate="G$1" x="182.88" y="469.9" smashed="yes"/>
-<instance part="GND34" gate="G$1" x="182.88" y="337.82" smashed="yes" rot="R90"/>
+<instance part="GND34" gate="G$1" x="205.74" y="325.12" smashed="yes"/>
 <instance part="GND45" gate="G$1" x="337.82" y="7.62" smashed="yes"/>
 <instance part="GND43" gate="G$1" x="335.28" y="30.48" smashed="yes"/>
@@
 <instance part="U200" gate="SUP" x="515.62" y="327.66"/>
 <instance part="SUPPLY41" gate="1" x="515.62" y="345.44" smashed="yes"/>
+<instance part="R101" gate="R" x="205.74" y="332.74" smashed="yes" rot="R90">
+<attribute name="NAME" x="208.28" y="332.74" size="1.778" layer="95"/>
+<attribute name="VALUE" x="208.28" y="330.2" size="1.778" layer="96"/>
+</instance>
 </instances>
 <busses>
@@
 </segment>
 <segment>
-<pinref part="GND34" gate="G$1" pin="GND"/>
-<pinref part="U100" gate="U" pin="BOOT1/FT/PB2"/>
-</segment>
-<segment>
 <pinref part="R400" gate="R" pin="1"/>
 <pinref part="GND5" gate="G$1" pin="GND"/>
@@
 <junction x="515.62" y="314.96"/>
 </segment>
+<segment>
+<pinref part="R101" gate="R" pin="1"/>
+<pinref part="GND34" gate="G$1" pin="GND"/>
+</segment>
 </net>
 <net name="3V3" class="0">
@@
 </segment>
 </net>
-<net name="MCU_AUX9" class="0">
+<net name="FSMC_A7" class="0">
 <segment>
 <pinref part="U700" gate="BANK2" pin="IOB_56"/>
@@
 </segment>
 </net>
-<net name="MCU_AUX10" class="0">
+<net name="FSMC_A10" class="0">
 <segment>
 <pinref part="U700" gate="BANK2" pin="IOB_57"/>
@@
 </segment>
 <segment>
-<pinref part="U100" gate="U" pin="PG1/FT/FSMC_A11"/>
-<wire x1="73.66" y1="340.36" x2="71.12" y2="340.36" width="0.1524" layer="91"/>
-<label x="71.12" y="340.36" size="1.778" layer="95" align="center-right"/>
+<pinref part="U100" gate="U" pin="PG0/FT/FSMC_A10"/>
+<wire x1="73.66" y1="342.9" x2="71.12" y2="342.9" width="0.1524" layer="91"/>
+<label x="71.12" y="342.9" size="1.778" layer="95" align="center-right"/>
 </segment>
 </net>
-<net name="MCU_AUX11" class="0">
+<net name="FSMC_A8" class="0">
 <segment>
 <pinref part="U700" gate="BANK2" pin="IOB_61"/>
@@
 </segment>
 </net>
-<net name="MCU_AUX12" class="0">
+<net name="FSMC_A9" class="0">
 <segment>
 <pinref part="U700" gate="BANK2" pin="IOB_63"/>
@@
 </segment>
 <segment>
-<pinref part="U100" gate="U" pin="FSMC_NIOS16/FT/PF11"/>
-<wire x1="180.34" y1="358.14" x2="182.88" y2="358.14" width="0.1524" layer="91"/>
-<label x="182.88" y="358.14" size="1.778" layer="95" align="center-left"/>
+<pinref part="U100" gate="U" pin="ADC12_IN14/PC4"/>
+<wire x1="180.34" y1="419.1" x2="182.88" y2="419.1" width="0.1524" layer="91"/>
+<label x="182.88" y="419.1" size="1.778" layer="95" align="center-left"/>
 </segment>
 </net>
@@
 </segment>
 <segment>
-<pinref part="U100" gate="U" pin="ADC12_IN9/TIM3_CH4('00'OR'10')/TIM8_CH3N/TIM1_CH3N('01')/PB1"/>
-<wire x1="180.34" y1="340.36" x2="182.88" y2="340.36" width="0.1524" layer="91"/>
-<label x="182.88" y="340.36" size="1.778" layer="95"/>
+<pinref part="U100" gate="U" pin="ADC12_IN15/PC5"/>
+<wire x1="180.34" y1="416.56" x2="182.88" y2="416.56" width="0.1524" layer="91"/>
+<label x="182.88" y="416.56" size="1.778" layer="95" align="center-left"/>
 </segment>
 </net>
@@
 </segment>
 </net>
-<net name="DISPLAY_AUX2" class="0">
+<net name="DISPLAY_AUX1" class="0">
 <segment>
-<pinref part="U100" gate="U" pin="ADC12_IN15/PC5"/>
-<wire x1="180.34" y1="416.56" x2="182.88" y2="416.56" width="0.1524" layer="91"/>
-<label x="182.88" y="416.56" size="1.778" layer="95" align="center-left"/>
+<pinref part="U100" gate="U" pin="ADC12_IN9/TIM3_CH4('00'OR'10')/TIM8_CH3N/TIM1_CH3N('01')/PB1"/>
+<wire x1="180.34" y1="340.36" x2="182.88" y2="340.36" width="0.1524" layer="91"/>
+<label x="182.88" y="340.36" size="1.778" layer="95"/>
 </segment>
 <segment>
@@
 </segment>
 </net>
-<net name="DISPLAY_AUX1" class="0">
-<segment>
-<pinref part="U100" gate="U" pin="ADC12_IN14/PC4"/>
-<wire x1="180.34" y1="419.1" x2="182.88" y2="419.1" width="0.1524" layer="91"/>
-<label x="182.88" y="419.1" size="1.778" layer="95" align="center-left"/>
-</segment>
-<segment>
-<pinref part="J4" gate="J" pin="5"/>
-<wire x1="711.2" y1="58.42" x2="706.12" y2="58.42" width="0.1524" layer="91"/>
-<label x="706.12" y="58.42" size="1.778" layer="95" align="center-right"/>
-</segment>
-</net>
 <net name="D-" class="0">
 <segment>
@@
 </segment>
 </net>
+<net name="DISPLAY_RESET" class="0">
+<segment>
+<pinref part="U100" gate="U" pin="BOOT1/FT/PB2"/>
+<pinref part="R101" gate="R" pin="2"/>
+<wire x1="180.34" y1="337.82" x2="205.74" y2="337.82" width="0.1524" layer="91"/>
+<wire x1="205.74" y1="337.82" x2="210.82" y2="337.82" width="0.1524" layer="91"/>
+<junction x="205.74" y="337.82"/>
+<label x="210.82" y="337.82" size="1.778" layer="95"/>
+</segment>
+<segment>
+<pinref part="J4" gate="J" pin="5"/>
+<wire x1="711.2" y1="58.42" x2="706.12" y2="58.42" width="0.1524" layer="91"/>
+<label x="706.12" y="58.42" size="1.778" layer="95" align="center-right"/>
+</segment>
+</net>
+<net name="N$10" class="0">
+<segment>
+<pinref part="U100" gate="U" pin="FSMC_NIOS16/FT/PF11"/>
+<wire x1="180.34" y1="358.14" x2="182.88" y2="358.14" width="0.1524" layer="91"/>
+</segment>
+</net>
+<net name="FSMC_A6" class="0">
+<segment>
+<pinref part="U100" gate="U" pin="FSMC_A6/FT/PF12"/>
+<wire x1="180.34" y1="355.6" x2="182.88" y2="355.6" width="0.1524" layer="91"/>
+<label x="182.88" y="355.6" size="1.778" layer="95"/>
+</segment>
+<segment>
+<pinref part="U700" gate="BANK2" pin="IOB_64"/>
+<wire x1="492.76" y1="58.42" x2="490.22" y2="58.42" width="0.1524" layer="91"/>
+<label x="490.22" y="58.42" size="1.778" layer="95" align="center-right"/>
+</segment>
+</net>
+<net name="MCU_INT2" class="0">
+<segment>
+<pinref part="U100" gate="U" pin="PG1/FT/FSMC_A11"/>
+<wire x1="73.66" y1="340.36" x2="71.12" y2="340.36" width="0.1524" layer="91"/>
+<label x="71.12" y="340.36" size="1.778" layer="95" align="center-right"/>
+</segment>
+<segment>
+<pinref part="U700" gate="BANK0" pin="IOT_171"/>
+<wire x1="391.16" y1="144.78" x2="388.62" y2="144.78" width="0.1524" layer="91"/>
+<label x="388.62" y="144.78" size="1.778" layer="95" align="center-right"/>
+</segment>
+</net>

Commit message: rewiring of v1c schematic continues
renamed MCU_AUX7 to MCU_INT0
renamed MCU_AUX8 to MCU_INT1
renamed MCU_INT0 to MCU_PWM0
renamed PWM to MCU_PWM1
moved LAT_OE to FPGA pin 96
moved LAT_DIR to FPGA pin 95
moved LAT_0 to FPGA pin 94
moved LAT_1 to FPGA pin 93
moved LAT_2 to FPGA pin 91
moved LAT_3 to FPGA pin 90
moved LAT_4 to FPGA pin 88
moved LAT_5 to FPGA pin 87
moved LAT_6 to FPGA pin 85
moved LAT_7 to FPGA pin 84
moved ADC_MUX S0 to FPGA pin 80
moved ADC_MUX S1 to FPGA pin 81
moved ADC_MUX S2 to FPGA pin 82
moved ADC_MUX S3 to FPGA pin 83
renamed DISPLAY_D/P to DISPLAY_AUX1
renamed DISPLAY_AUX2 to DISPLAY_D/P
added 220R series resistors to each BPIOs
wired ADC_MUX_EN to FPGA pin 55, since pin 114 is already MCU_INT2
Parts:
- added R424, R425, R426, R427, R428, R429, R430, R431: 220R, dp_devices.v6:RESISTOR-0402
Connections:
- net PWM renamed MCU_PWM1
- removed net MCU_AUX7: U100U.PE0/FT/TIM4_ETR/FSMC_NBL0, U700BANK0.IOT_191
- removed net MCU_AUX8: U100U.PE1/FT/FSMC_NBL1, U700BANK0.IOT_190
- new net BPIO0I: R404.2, R424.2, U400.B, U402G.O
- new net BPIO1I: R410.2, R425.2, U404.B, U406G.O
- new net BPIO2I: R416.2, R426.2, U408.B, U410G.O
- new net BPIO3I: R422.2, R427.2, U412.B, U414G.O
- new net BPIO4I: R405.2, R428.2, U401.B, U403G.O
- new net BPIO5I: R411.2, R429.2, U405.B, U407G.O
- new net BPIO6I: R417.2, R430.2, U409.B, U411G.O
- new net BPIO7I: R423.2, R431.2, U413.B, U415G.O
- new net MCU_INT1I: U100U.TIM8_CH4/TIM3_CH4('11')/FT/PC9, U700BANK0.IOT_172
- new net MCU_PWM0: U100U.PA10/FT/USART1_RX('0')/TIM1_CH3('00'OR'01'), U700BANK0.GBIN0/IOT_198
- net ADC_MUX_EN: now also U700BANK2.IOB_91; no longer U700BANK1.IOR_146
- net ADC_MUX_S0: now also U700BANK1.IOR_116; no longer U700BANK1.GBIN3/IOR_140
- net ADC_MUX_S1: now also U700BANK1.IOR_117; no longer U700BANK1.GBIN2/IOR_141
- net ADC_MUX_S2: now also U700BANK1.IOR_118; no longer U700BANK1.IOR_144
- net ADC_MUX_S3: now also U700BANK1.IOR_119
- net BPIO0: now also R424.1; no longer R404.2, U400.B, U402G.O
- net BPIO1: now also R425.1; no longer R410.2, U404.B, U406G.O
- net BPIO2: now also R426.1; no longer R416.2, U408.B, U410G.O
- net BPIO3: now also R427.1; no longer R422.2, U412.B, U414G.O
- net BPIO4: now also R428.1; no longer R405.2, U401.B, U403G.O
- net BPIO5: now also R429.1; no longer R411.2, U405.B, U407G.O
- net BPIO6: now also R430.1; no longer R417.2, U409.B, U411G.O
- net BPIO7: now also R431.1; no longer R423.2, U413.B, U415G.O
- net DISPLAY_AUX1: now also J4.2; no longer J4.4
- net DISPLAY_CS: now also U100U.FSMC_NIOS16/FT/PF11; no longer U100U.ADC12_IN14/PC4
- net DISPLAY_D/P: now also J4.4; no longer J4.2
- net LAT0: now also U700BANK1.GBIN2/IOR_141; no longer U700BANK1.IOR_139
- net LAT1: now also U700BANK1.GBIN3/IOR_140; no longer U700BANK1.IOR_138
- net LAT2: now also U700BANK1.IOR_139; no longer U700BANK1.IOR_137
- net LAT3: now also U700BANK1.IOR_138; no longer U700BANK1.IOR_136
- net LAT4: now also U700BANK1.IOR_137; no longer U700BANK1.IOR_128
- net LAT5: now also U700BANK1.IOR_136; no longer U700BANK1.IOR_120
- net LAT6: now also U700BANK1.IOR_128; no longer U700BANK1.IOR_119
- net LAT7: now also U700BANK1.IOR_120; no longer U700BANK1.IOR_118
- net LAT_DIR: now also U700BANK1.IOR_144; no longer U700BANK1.IOR_117
- net LAT_OE: now also U700BANK1.IOR_146; no longer U700BANK1.IOR_116
- net MCU_INT0: now also U100U.PE0/FT/TIM4_ETR/FSMC_NBL0, U700BANK0.IOT_191; no longer U100U.PA10/FT/USART1_RX('0')/TIM1_CH3('00'OR'01'), U700BANK0.GBIN0/IOT_198
- net MCU_INT1: now also U100U.PE1/FT/FSMC_NBL1, U700BANK0.IOT_190; no longer U100U.TIM8_CH4/TIM3_CH4('11')/FT/PC9, U700BANK0.IOT_172
- net N$10: now also U100U.ADC12_IN14/PC4; no longer U100U.FSMC_NIOS16/FT/PF11
Other:
- note added: "Need to connect ADC_MUX_EN to FPGA"
- note removed: "Need to connect ADC_MUX_S3 to FPGA"
