File: BPUv1c/BusPirate-ultra.v1.0c.sch (EAGLE design)
At the start: 193 parts, among them J1 USB-C-12, J2 CON_HEADER_1X04, J3 CON_HEADER_1X10-RIGHT_ANGLED_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, J4 CON_MOLEX_MALE_SMT_SH_1.25, Q300 PMV65XP, Q301 DMMT3906W, U100 STM32F103ZX, U101 W25X40CL, U200 74HCT4067, U201 MCP6001, U202 ADS7041, U300 MCP1824_ADJ, U301 MCP6001, U302 MCP1700, U303 MCP1801T-1202I/OT, U400 SN74LVC1T45DBV, U401 SN74LVC1T45DBV, U402 74LVC1G07DBV, U403 74LVC1G07DBV, U404 SN74LVC1T45DBV, U405 SN74LVC1T45DBV, U406 74LVC1G07DBV, U407 74LVC1G07DBV, U408 SN74LVC1T45DBV, U409 SN74LVC1T45DBV, U410 74LVC1G07DBV, U411 74LVC1G07DBV, U412 SN74LVC1T45DBV, U413 SN74LVC1T45DBV, U414 74LVC1G07DBV, U415 74LVC1G07DBV, U500 74HCT4066PW, U501 74HCT4066PW, U600 23LC1024, U601 23LC1024, U602 74LVC245A, U700 ICE40HX4K

Commit message: continued on v1c schematic changes renamed MCU_AUX4 to MCU_INT3 and move it from MCU PD6 to PD2 renamed MCU_INT1I to MCU_AUX0 fix display connections
Connections:
- net MCU_INT1I renamed MCU_AUX0
- removed net MCU_AUX4: U100U.PD6/FT/FSMC_NWAIT/USART2_RX('1'), U700BANK0.IOT_212
- removed net N$10: U100U.ADC12_IN14/PC4
- removed net N$29: U100U.PD2/FT/TIM3_ETR/UART5_RX
- new net DISPLAY_CSI: U100U.FSMC_NIOS16/FT/PF11
- new net MCU_INT3: U100U.PD2/FT/TIM3_ETR/UART5_RX, U700BANK0.IOT_212
- net DISPLAY_CS: now also J4.5, U100U.ADC12_IN14/PC4; no longer J4.1, U100U.FSMC_NIOS16/FT/PF11
- net DISPLAY_RESET: now also J4.1; no longer J4.5
Changed lines of the file:
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@@
 </segment>
 </net>
-<net name="MCU_INT1I" class="0">
+<net name="MCU_AUX0" class="0">
 <segment>
 <pinref part="U700" gate="BANK0" pin="IOT_172"/>
@@
 </segment>
 </net>
-<net name="MCU_AUX4" class="0">
-<segment>
-<pinref part="U100" gate="U" pin="PD6/FT/FSMC_NWAIT/USART2_RX('1')"/>
-<wire x1="73.66" y1="414.02" x2="71.12" y2="414.02" width="0.1524" layer="91"/>
-<label x="71.12" y="414.02" size="1.778" layer="95" align="center-right"/>
-</segment>
+<net name="MCU_INT3" class="0">
 <segment>
 <pinref part="U700" gate="BANK0" pin="IOT_212"/>
 <wire x1="426.72" y1="157.48" x2="431.8" y2="157.48" width="0.1524" layer="91"/>
 <label x="431.8" y="157.48" size="1.778" layer="95" align="center-left"/>
+</segment>
+<segment>
+<pinref part="U100" gate="U" pin="PD2/FT/TIM3_ETR/UART5_RX"/>
+<wire x1="73.66" y1="424.18" x2="71.12" y2="424.18" width="0.1524" layer="91"/>
+<label x="71.12" y="424.18" size="1.778" layer="95" align="center-right"/>
 </segment>
 </net>
@@
 <wire x1="73.66" y1="464.82" x2="71.12" y2="464.82" width="0.1524" layer="91"/>
 <label x="71.12" y="464.82" size="1.778" layer="95" align="center-right"/>
-</segment>
-</net>
-<net name="N$29" class="0">
-<segment>
-<pinref part="U100" gate="U" pin="PD2/FT/TIM3_ETR/UART5_RX"/>
-<wire x1="73.66" y1="424.18" x2="71.12" y2="424.18" width="0.1524" layer="91"/>
 </segment>
 </net>
@@
 </segment>
 </net>
-<net name="DISPLAY_CS" class="0">
-<segment>
-<pinref part="J4" gate="J" pin="1"/>
-<wire x1="711.2" y1="68.58" x2="706.12" y2="68.58" width="0.1524" layer="91"/>
-<label x="706.12" y="68.58" size="1.778" layer="95" align="center-right"/>
-</segment>
-<segment>
-<pinref part="U100" gate="U" pin="FSMC_NIOS16/FT/PF11"/>
-<wire x1="180.34" y1="358.14" x2="182.88" y2="358.14" width="0.1524" layer="91"/>
-<label x="182.88" y="358.14" size="1.778" layer="95"/>
-</segment>
-</net>
 <net name="DISPLAY_AUX1" class="0">
 <segment>
@@
 </segment>
 </net>
-<net name="DISPLAY_RESET" class="0">
-<segment>
-<pinref part="U100" gate="U" pin="BOOT1/FT/PB2"/>
-<pinref part="R101" gate="R" pin="2"/>
-<wire x1="180.34" y1="337.82" x2="205.74" y2="337.82" width="0.1524" layer="91"/>
-<wire x1="205.74" y1="337.82" x2="210.82" y2="337.82" width="0.1524" layer="91"/>
-<junction x="205.74" y="337.82"/>
-<label x="210.82" y="337.82" size="1.778" layer="95"/>
-</segment>
+<net name="DISPLAY_CS" class="0">
 <segment>
 <pinref part="J4" gate="J" pin="5"/>
 <wire x1="711.2" y1="58.42" x2="706.12" y2="58.42" width="0.1524" layer="91"/>
 <label x="706.12" y="58.42" size="1.778" layer="95" align="center-right"/>
+</segment>
+<segment>
+<pinref part="U100" gate="U" pin="ADC12_IN14/PC4"/>
+<wire x1="180.34" y1="419.1" x2="182.88" y2="419.1" width="0.1524" layer="91"/>
+<label x="182.88" y="419.1" size="1.778" layer="95"/>
 </segment>
 </net>
@@
 </segment>
 </net>
-<net name="N$10" class="0">
-<segment>
-<pinref part="U100" gate="U" pin="ADC12_IN14/PC4"/>
-<wire x1="180.34" y1="419.1" x2="182.88" y2="419.1" width="0.1524" layer="91"/>
-</segment>
-</net>
+<net name="DISPLAY_CSI" class="0">
+<segment>
+<pinref part="U100" gate="U" pin="FSMC_NIOS16/FT/PF11"/>
+<wire x1="180.34" y1="358.14" x2="182.88" y2="358.14" width="0.1524" layer="91"/>
+<label x="182.88" y="358.14" size="1.778" layer="95"/>
+</segment>
+</net>
+<net name="DISPLAY_RESET" class="0">
+<segment>
+<pinref part="J4" gate="J" pin="1"/>
+<wire x1="711.2" y1="68.58" x2="706.12" y2="68.58" width="0.1524" layer="91"/>
+<label x="706.12" y="68.58" size="1.778" layer="95" align="center-right"/>
+</segment>
+<segment>
+<pinref part="U100" gate="U" pin="BOOT1/FT/PB2"/>
+<pinref part="R101" gate="R" pin="2"/>
+<wire x1="180.34" y1="337.82" x2="205.74" y2="337.82" width="0.1524" layer="91"/>
+<wire x1="205.74" y1="337.82" x2="210.82" y2="337.82" width="0.1524" layer="91"/>
+<junction x="205.74" y="337.82"/>
+<label x="210.82" y="337.82" size="1.778" layer="95"/>
+</segment>
+</net>
